Commit message: head fix.

File: velma_defs/defs/head.urdf.xacro (robot description, xacro)
@@ -28,14 +28,7 @@
     </joint>
     <link name="head_tilt_link"/>
-    <joint name="head_plate_joint" type="fixed">
-      <origin xyz="0 -0.03 0.0" rpy="1.57 0 0"/>
+    <joint name="stereo_left_joint" type="fixed">
+      <origin xyz="0 -0.205 -0.045" rpy="1.57.0 0 0"/>
       <parent link="head_tilt_link"/>
-      <child link="head_plate_link"/>
-    </joint>
-    <link name="head_plate_link">
-    </link>
-    <joint name="stereo_left_joint" type="fixed">
-      <origin xyz="0 0.045 0.175 " rpy="0.0 0 0"/>
-      <parent link="head_plate_link"/>
       <child link="stereo_left_link"/>
     </joint>
@@ -43,5 +36,5 @@
     </link>
     <joint name="stereo_right_joint" type="fixed">
-      <origin xyz="0 -0.09 0.0" rpy="0.0 0 0"/>
+      <origin xyz="0 -0.09 0.0" rpy="0 0 0"/>
       <parent link="stereo_left_link"/>
       <child link="stereo_right_link"/>

Commit message: head defs.

File: velma_defs/defs/head.urdf.xacro (robot description, xacro)
@@ -1,4 +1,5 @@
 <?xml version="1.0"?>
 <robot>
+  <include filename="$(find velma_defs)/defs/camera.urdf.xacro" />
   <macro name="velma_head" params="parent *origin">
     <joint name="head_frame_joint" type="fixed">
@@ -28,18 +29,23 @@
     </joint>
     <link name="head_tilt_link"/>
-    <joint name="stereo_left_joint" type="fixed">
-      <origin xyz="0 -0.205 -0.045" rpy="1.57.0 0 0"/>
-      <parent link="head_tilt_link"/>
-      <child link="stereo_left_link"/>
-    </joint>
-    <link name="stereo_left_link">
-    </link>
-    <joint name="stereo_right_joint" type="fixed">
-      <origin xyz="0 -0.09 0.0" rpy="0 0 0"/>
-      <parent link="stereo_left_link"/>
-      <child link="stereo_right_link"/>
-    </joint>
-    <link name="stereo_right_link">
-    </link>
+    <!-- sensors -->
+    <head_camera parent="head_tilt_link" name="stereo_left">
+      <origin xyz="0.074819 -0.19424 0.039144" rpy="1.572 -0.0046408 0.0147"/>
+    </head_camera>
+    <head_camera parent="stereo_left_link" name="stereo_right">
+      <origin xyz="0.0 -0.09 0.0" rpy="0 0 0"/>
+    </head_camera>
+    <head_camera parent="stereo_left_link" name="kinect_left_rgb">
+      <origin xyz="0.013309 -0.010124 -0.06841" rpy="1.5634 -0.022662 0.37293"/>
+    </head_camera>
+    <head_camera parent="kinect_left_rgb_link" name="kinect_left_ir">
+      <origin xyz="0.0 0.03 0.0" rpy="0 0 0"/>
+    </head_camera>
+    <head_camera parent="stereo_left_link" name="kinect_right_rgb">
+      <origin xyz="0.00045739 -0.071104 -0.074766" rpy="1.5892 -0.035955 -0.34978"/>
+    </head_camera>
+    <head_camera parent="kinect_right_rgb_link" name="kinect_right_ir">
+      <origin xyz="0.0 0.03 0.0" rpy="0 0 0"/>
+    </head_camera>
   </macro>
 </robot>

Commit message: new calubration

File: velma_defs/defs/head.urdf.xacro (robot description, xacro)
@@ -16,5 +16,5 @@
       <parent link="head_frame"/>
       <child link="head_pan_link"/>
-      <limit effort="100" velocity="100"/>
+      <limit lower="-1.57" upper="1.57" effort="100" velocity="100"/>
     </joint>
     <link name="head_pan_link">
@@ -22,26 +22,35 @@
     <!-- tilt -->
     <joint name="head_tilt_joint" type="revolute">
-      <origin xyz="0 0 0.05" rpy="-1.57 0.0 0" />
+      <origin xyz="0 0 0.0" rpy="-1.57 0.0 0" />
       <axis xyz="0 0 1"/>
       <parent link="head_pan_link"/>
       <child link="head_tilt_link"/>
-      <limit effort="100" velocity="100"/>
+      <limit lower="-1.57" upper="1.57" effort="100" velocity="100"/>
     </joint>
     <link name="head_tilt_link"/>
     <!-- sensors -->
     <head_camera parent="head_tilt_link" name="stereo_left">
-      <origin xyz="0.074819 -0.19424 0.039144" rpy="1.572 -0.0046408 0.0147"/>
+      <!--<origin xyz="0.074819 -0.19424 0.039144" rpy="1.572 -0.0046408 0.0147"/> -->
+      <!-- <origin xyz="0.072474    -0.21002    0.043726" rpy="1.5767  -0.0094749   0.0058925"/> -->
+      <origin xyz="${cal_head_to_stereo_left_x} ${cal_head_to_stereo_left_y} ${cal_head_to_stereo_left_z}"
+              rpy="${cal_head_to_stereo_left_roll} ${cal_head_to_stereo_left_pitch} ${cal_head_to_stereo_left_yaw}"/>
     </head_camera>
     <head_camera parent="stereo_left_link" name="stereo_right">
       <origin xyz="0.0 -0.09 0.0" rpy="0 0 0"/>
     </head_camera>
-    <head_camera parent="stereo_left_link" name="kinect_left_rgb">
-      <origin xyz="0.013309 -0.010124 -0.06841" rpy="1.5634 -0.022662 0.37293"/>
+    <head_camera parent="head_tilt_link" name="kinect_left_rgb">
+      <!--<origin xyz="0.013309 -0.010124 -0.06841" rpy="1.5634 -0.022662 0.37293"/> -->
+      <!--<origin xyz="0.019408   -0.010485   -0.088064" rpy="1.5637  -0.0097296     0.36447"/>-->
+      <origin xyz="${cal_stereo_left_to_kinect_left_x} ${cal_stereo_left_to_kinect_left_y} ${cal_stereo_left_to_kinect_left_z}"
+              rpy="${cal_stereo_left_to_kinect_left_roll} ${cal_stereo_left_to_kinect_left_pitch} ${cal_stereo_left_to_kinect_left_yaw}"/>
     </head_camera>
     <head_camera parent="kinect_left_rgb_link" name="kinect_left_ir">
       <origin xyz="0.0 0.03 0.0" rpy="0 0 0"/>
     </head_camera>
-    <head_camera parent="stereo_left_link" name="kinect_right_rgb">
-      <origin xyz="0.00045739 -0.071104 -0.074766" rpy="1.5892 -0.035955 -0.34978"/>
+    <head_camera parent="head_tilt_link" name="kinect_right_rgb">
+      <!--<origin xyz="0.00045739 -0.071104 -0.074766" rpy="1.5892 -0.035955 -0.34978"/> -->
+      <!--<origin xyz="-0.034936    -0.05614   -0.084153" rpy="1.588   -0.024981    -0.37211"/>-->
+      <origin xyz="${cal_stereo_left_to_kinect_right_x} ${cal_stereo_left_to_kinect_right_y} ${cal_stereo_left_to_kinect_right_z}"
+              rpy="${cal_stereo_left_to_kinect_right_roll} ${cal_stereo_left_to_kinect_right_pitch} ${cal_stereo_left_to_kinect_right_yaw}"/>
     </head_camera>
     <head_camera parent="kinect_right_rgb_link" name="kinect_right_ir">
