Commit message: urdf fix.

File: velma_defs/robots/velma.urdf.xacro (robot description, xacro)
@@ -32,5 +32,5 @@
   <joint name="torso_1_joint" type="revolute">
     <origin xyz="0 0 0.80" rpy="${M_PI/2} 0 0"/>
-    <axis xyz="0 0 1"/>
+    <axis xyz="0 0 -1"/>
     <limit lower="${M_PI/4}" upper="${105 * M_PI/180}" effort="100" velocity="100"/>
     <parent link="torso_link0"/>
@@ -41,5 +41,5 @@
   <joint name="torso_2_joint" type="revolute">
     <origin xyz="0.375 0 0" rpy="0 0 0"/>
-    <axis xyz="0 0 1"/>
+    <axis xyz="0 0 -1"/>
     <limit lower="-1.57" upper="1.57" effort="100" velocity="100"/>
     <mimic joint="torso_1_joint" multiplier="-1"/>

Commit message: updated bringup scripts

File: velma_defs/robots/velma.urdf.xacro (robot description, xacro)
@@ -8,6 +8,6 @@
   <include filename="$(find lwr_defs)/defs/kuka_lwr_arm_defs.xml"/>
   <include filename="$(find lwr_defs)/defs/materials.xml"/>
-  <!--
-  <include filename="$(find barret_hand_defs)/defs/barret_hand.urdf.xacro"/>
+  <include filename="$(find barrett_hand_defs)/defs/barret_hand.urdf.xacro"/>
+<!--
   <include filename="$(find velma_defs)/defs/kinect_camera.urdf.xacro" />
   <include filename="$(find velma_defs)/defs/head.urdf.xacro" /> -->
@@ -55,4 +55,10 @@
     <origin xyz="0 0.1641 -0.07943" rpy="${-5*M_PI/6} 0 0"/>
   </kuka_lwr_arm>
+  <xacro:barret_hand prefix="right" parent="right_arm_7_link">
+    <origin xyz="0.115 0.0 -0.055" rpy="0 ${M_PI/2} 0"/>
+  </xacro:barret_hand>
+  <xacro:barret_hand prefix="left" parent="left_arm_7_link">
+    <origin xyz="-0.115 0.0 -0.055" rpy="0 ${-M_PI/2} 0"/>
+  </xacro:barret_hand>
 <!--
   <joint name="torso_right_arm_joint" type="fixed">

Commit message: Add visualization models.

File: velma_defs/robots/velma.urdf.xacro (robot description, xacro)
@@ -48,4 +48,11 @@
   </joint>
   <link name="torso_link2">
+    <visual>
+      <origin xyz="0 0.04 0" rpy="${-M_PI/2.0} 0 0.0" />
+      <!--origin xyz="-0.03 -0.07 0" rpy="0 0 -1.57"-->
+      <geometry>
+        <mesh filename="package://velma_description/meshes/arm_base.STL" />
+      </geometry>
+    </visual>
   </link>
   <kuka_lwr_arm parent="torso_link2" name="right" right="1">
@@ -55,25 +62,35 @@
     <origin xyz="0 0.1641 -0.07943" rpy="${-5*M_PI/6} 0 0"/>
   </kuka_lwr_arm>
+  <joint name="right_gripper_mount_joint" type="fixed">
+    <origin xyz="0 0 0" rpy="0 0 0"/>
+    <parent link="right_arm_7_link"/>
+    <child link="right_gripper_mount_link"/>
+  </joint>
+  <link name="right_gripper_mount_link">
+    <visual>
+      <origin xyz="0 0 0" rpy="0.0 0 0" />
+      <geometry>
+        <mesh filename="package://velma_description/meshes/gripper_mount.STL" />
+      </geometry>
+    </visual>
+  </link>
+  <joint name="left_gripper_mount_joint" type="fixed">
+    <origin xyz="0 0 0" rpy="0 0 ${M_PI}"/>
+    <parent link="left_arm_7_link"/>
+    <child link="left_gripper_mount_link"/>
+  </joint>
+  <link name="left_gripper_mount_link">
+    <visual>
+      <origin xyz="0 0 0" rpy="0.0 0 0" />
+      <geometry>
+        <mesh filename="package://velma_description/meshes/gripper_mount.STL" />
+      </geometry>
+    </visual>
+  </link>
   <xacro:barret_hand prefix="right" parent="right_arm_7_link">
-    <origin xyz="0.115 0.0 -0.055" rpy="0 ${M_PI/2} 0"/>
+    <origin xyz="0.115 0.0 -0.078" rpy="0 ${M_PI/2} 0"/>
   </xacro:barret_hand>
   <xacro:barret_hand prefix="left" parent="left_arm_7_link">
-    <origin xyz="-0.115 0.0 -0.055" rpy="0 ${-M_PI/2} 0"/>
+    <origin xyz="-0.115 0.0 -0.078" rpy="0 ${-M_PI/2} 0"/>
   </xacro:barret_hand>
-<!--
-  <joint name="torso_right_arm_joint" type="fixed">
-    <origin xyz="0 0.0941 0.07943" rpy="${-M_PI/6} 0 0"/>
-    <parent link="torso_link2"/>
-    <child link="torso_right_arm_base"/>
-  </joint>
-  <link name="torso_right_arm_base">
-  </link>
-  <joint name="torso_left_arm_joint" type="fixed">
-    <origin xyz="0 0.0941 -0.07943" rpy="${-5 * M_PI/6} 0 0"/>
-    <parent link="torso_link2"/>
-    <child link="torso_left_arm_base"/>
-  </joint>
-  <link name="torso_left_arm_base">
-  </link>
--->
 </robot>

Commit message: fix deprecated include in xacro.

File: velma_defs/robots/velma.urdf.xacro (robot description, xacro)
@@ -5,13 +5,13 @@
                         xmlns:xacro="http://playerstage.sourceforge.net/gazebo/xmlschema/#interface"
 	 name="velma">
-  <include filename="$(find velma_description)/calibration/default_cal.xml"/>
-  <include filename="$(find lwr_defs)/defs/kuka_lwr_arm_defs.xml"/>
-  <include filename="$(find lwr_defs)/defs/materials.xml"/>
-  <include filename="$(find barrett_hand_defs)/defs/barret_hand.urdf.xacro"/>
+  <xacro:include filename="$(find velma_description)/calibration/default_cal.xml"/>
+  <xacro:include filename="$(find lwr_defs)/defs/kuka_lwr_arm_defs.xml"/>
+  <xacro:include filename="$(find lwr_defs)/defs/materials.xml"/>
+  <xacro:include filename="$(find barrett_hand_defs)/defs/barret_hand.urdf.xacro"/>
 <!--
   <include filename="$(find velma_defs)/defs/kinect_camera.urdf.xacro" />
   <include filename="$(find velma_defs)/defs/head.urdf.xacro" /> -->
-<property name="M_PI" value="3.1415926535897931" />
-<link name="world" />
+  <property name="M_PI" value="3.1415926535897931" />
+  <link name="world" />
   <joint name="arm_world_joint" type="fixed">
     <origin xyz="0 0 0.1" rpy="0 0 0"/>
