Commit message: jade support

File: velma_description/defs/camera.urdf.xacro (robot description, xacro)
@@ -1,8 +1,11 @@
 <?xml version="1.0"?>
-<robot>
-  <macro name="head_camera" params="name parent *origin">
+<robot xmlns:controller="http://playerstage.sourceforge.net/gazebo/xmlschema/#controller"
+                        xmlns:interface="http://playerstage.sourceforge.net/gazebo/xmlschema/#interface"
+                        xmlns:sensor="http://playerstage.sourceforge.net/gazebo/xmlschema/#sensor"
+                        xmlns:xacro="http://www.ros.org/wiki/xacro">
+  <xacro:macro name="head_camera" params="name parent *origin">
     <!-- sensor physical attachment -->
     <joint name="${name}_joint" type="fixed">
-      <insert_block name="origin" />
+      <xacro:insert_block name="origin" />
       <parent link="${parent}"/>
       <child link="${name}_link"/>
@@ -16,4 +19,4 @@
     </joint>
     <link name="${name}_optical_frame"/>
-  </macro>
+  </xacro:macro>
 </robot>

File: velma_description/defs/head.urdf.xacro (robot description, xacro)
@@ -3,9 +3,9 @@
                         xmlns:interface="http://playerstage.sourceforge.net/gazebo/xmlschema/#interface"
                         xmlns:sensor="http://playerstage.sourceforge.net/gazebo/xmlschema/#sensor"
-                        xmlns:xacro="http://playerstage.sourceforge.net/gazebo/xmlschema/#interface">
+                        xmlns:xacro="http://www.ros.org/wiki/xacro">
   <xacro:include filename="$(find velma_description)/defs/camera.urdf.xacro" />
-  <macro name="velma_head" params="parent *origin">
+  <xacro:macro name="velma_head" params="parent *origin">
     <joint name="head_base_joint" type="fixed">
-      <insert_block name="origin" />
+      <xacro:insert_block name="origin" />
       <parent link="${parent}"/>
       <child link="head_base"/>
@@ -165,4 +165,4 @@
               rpy="${cal_head_kinect_rgb_joint_roll} ${cal_head_kinect_rgb_joint_pitch} ${cal_head_kinect_rgb_joint_yaw}"/>
     </head_camera>
-  </macro>
+  </xacro:macro>
 </robot>

File: velma_description/defs/kinect_camera.urdf.xacro (robot description, xacro)
@@ -1,7 +1,7 @@
 <?xml version="1.0"?>
 <robot>
-  <macro name="kinect_camera" params="name parent *origin">
+  <xacro:macro name="kinect_camera" params="name parent *origin">
     <joint name="${name}_frame_joint" type="fixed">
-      <insert_block name="origin" />
+      <xacro:insert_block name="origin" />
       <parent link="${parent}"/>
       <child link="${name}_frame"/>
@@ -65,4 +65,4 @@
     </joint>
     <link name="${name}_rgb_optical_frame"/>
-  </macro>
+  </xacro:macro>
 </robot>

File: velma_description/defs/torso.urdf.xacro (robot description, xacro)
@@ -1,7 +1,10 @@
 <?xml version="1.0"?>
-<robot>
-  <macro name="velma_torso" params="parent *origin">
+<robot xmlns:controller="http://playerstage.sourceforge.net/gazebo/xmlschema/#controller"
+                        xmlns:interface="http://playerstage.sourceforge.net/gazebo/xmlschema/#interface"
+                        xmlns:sensor="http://playerstage.sourceforge.net/gazebo/xmlschema/#sensor"
+                        xmlns:xacro="http://www.ros.org/wiki/xacro">
+  <xacro:macro name="velma_torso" params="parent *origin">
     <joint name="torso_base_joint" type="fixed">
-      <insert_block name="origin" />
+      <xacro:insert_block name="origin" />
       <parent link="${parent}"/>
       <child link="torso_base"/>
@@ -89,4 +92,4 @@
       </inertial>
     </link>
-  </macro>
+  </xacro:macro>
 </robot>

File: velma_description/robots/torso.urdf.xacro (robot description, xacro)
@@ -5,10 +5,10 @@
                         xmlns:xacro="http://playerstage.sourceforge.net/gazebo/xmlschema/#interface"
 	 name="torso">
-  <include filename="$(find velma_description)/calibration/default_cal.xml"/>
+  <xacro:include filename="$(find velma_description)/calibration/default_cal.xml"/>
 <!--
-  <include filename="$(find velma_defs)/defs/kinect_camera.urdf.xacro" />
+  <xacro:include filename="$(find velma_defs)/defs/kinect_camera.urdf.xacro" />
   -->
-  <include filename="$(find velma_description)/defs/head.urdf.xacro" />
-<property name="M_PI" value="3.1415926535897931" />
+  <xacro:include filename="$(find velma_description)/defs/head.urdf.xacro" />
+<xacro:property name="M_PI" value="3.1415926535897931" />
 <link name="world" />
   <joint name="arm_world_joint" type="fixed">

File: velma_description/robots/velma.urdf.xacro (robot description, xacro)
@@ -3,5 +3,5 @@
                         xmlns:interface="http://playerstage.sourceforge.net/gazebo/xmlschema/#interface"
                         xmlns:sensor="http://playerstage.sourceforge.net/gazebo/xmlschema/#sensor"
-                        xmlns:xacro="http://playerstage.sourceforge.net/gazebo/xmlschema/#interface"
+                        xmlns:xacro="http://www.ros.org/wiki/xacro"
 	 name="velma">
   <xacro:arg name="collision_model_full" default="true"/>
@@ -10,5 +10,5 @@
   <xacro:arg name="collision_model_no_hands" default="false"/>
   <xacro:arg name="gazebo_script" default="false"/>
-  <xacro:arg name="gazebo_ops_file"/>
+  <xacro:arg name="gazebo_ops_file" default=""/>
   <xacro:arg name="use_gazebo_kinect" default="false"/>
   <xacro:include filename="$(find velma_description)/calibration/default_cal.xml"/>
@@ -19,7 +19,7 @@
   <xacro:include filename="$(find barrett_hand_defs)/defs/barret_hand.urdf.xacro"/>
 <!--
-  <include filename="$(find velma_defs)/defs/kinect_camera.urdf.xacro" />
+  <xacro:include filename="$(find velma_defs)/defs/kinect_camera.urdf.xacro" />
    -->
-  <property name="camera_name" value="head_kinect" />
+  <xacro:property name="camera_name" value="head_kinect" />
   <!-- Gazebo Plugin -->
   <gazebo>
@@ -113,5 +113,5 @@
     </gazebo>
   </xacro:if>
-  <property name="M_PI" value="3.1415926535897931" />
+  <xacro:property name="M_PI" value="3.1415926535897931" />
   <link name="world" />
   <!-- static connection between the world frame and the map frame -->
