Commit message: torso stl fix

File: velma_description/defs/monokl.urdf.xacro (robot description, xacro)
@@ -64,5 +64,5 @@
       <sensor type="gpu_ray" name="${name}">
       <pose>0 0 0 0 0 0</pose>
-      <visualize>true</visualize>
+      <visualize>false</visualize>
       <update_rate>40</update_rate>
       <ray>

File: velma_description/defs/torso.urdf.xacro (robot description, xacro)
@@ -8,110 +8,4 @@
       <inertia ixx="${m*(3*r*r+h*h)/12}" ixy="0" ixz="0" iyy="${m*r*r/2}" iyz="0" izz="${m*(3*r*r+h*h)/12}" />
     </xacro:macro>
-   <!--  <gazebo>
-      <plugin name="gazebo_ros_control" filename="libgazebo_ros_control.so">
-        <robotNamespace>/</robotNamespace>
-      </plugin>
-    </gazebo>
-    <link name="omnitorso_y">
-      <inertial>
-        <mass value="0.001"/>
-        <inertia ixx="0" ixy="0" ixz="0" iyy="0" iyz="0" izz="0"/>
-      </inertial>
-      <collision>
-        <origin xyz="-0.081 0 0.1225" rpy="0.0 0 0" />
-        <geometry>
-          <mesh filename="package://omnivelma/meshes/collider/base.dae" />
-        </geometry>
-      </collision>
-      <visual>
-        <geometry>
-          <box size="0.364 0.32 0.15" />
-        </geometry>
-        <origin xyz="-0.035 0 0.25" rpy="0.0 0 0" />
-        <material name="torso_base">
-          <color rgba="0.3 0.3 0.15 1"/>
-        </material>
-      </visual>
-    </link>
-    <link name="omnitorso_x">
-      <inertial>
-        <mass value="0.001"/>
-        <inertia ixx="0" ixy="0" ixz="0" iyy="0" iyz="0" izz="0"/>
-      </inertial>
-      <collision>
-        <origin xyz="-0.081 0 0.1225" rpy="0.0 0 0" />
-        <geometry>
-          <mesh filename="package://omnivelma/meshes/collider/base.dae" />
-        </geometry>
-      </collision>
-      <visual>
-        <geometry>
-          <box size="0.364 0.32 0.15" />
-        </geometry>
-        <origin xyz="-0.035 0 0.25" rpy="0.0 0 0" />
-        <material name="torso_base">
-          <color rgba="0.3 0.3 0.15 1"/>
-        </material>
-      </visual>
-    </link>
-    <joint name="torso_base_joint" type="revolute">
-      <xacro:insert_block name="origin" />
-      <limit lower="-20.0" upper="20.0" effort="1000" velocity="1"/>
-      <axis xyz="0 0 1"/>
-      <parent link="${parent}"/>
-      <child link="omnitorso_x"/>
-    </joint>
-    <joint name="omni_joint_y" type="prismatic">
-      <origin xyz="0 0 0" rpy="0 0 0" />
-      <limit lower="-20.0" upper="20.0" effort="1000" velocity="1"/>
-      <axis xyz="0 1 0"/>
-      <parent link="omnitorso_x"/>
-      <child link="omnitorso_y"/>
-    </joint>
-    <joint name="omni_joint_x" type="prismatic">
-      <origin xyz="0 0 0" rpy="0 0 0" />
-      <limit lower="-20.0" upper="20.0" effort="1000" velocity="1"/>
-      <axis xyz="1 0 0"/>
-      <parent link="omnitorso_y"/>
-      <child link="torso_base"/>
-    </joint>
-    <transmission name="trans_rot">
-      <type>transmission_interface/SimpleTransmission</type>
-      <actuator name="$torso_base_motor">
-        <mechanicalReduction>1</mechanicalReduction>
-      </actuator>
-      <joint name="torso_base_joint">
-        <hardwareInterface>hardware_interface/PositionJointInterface</hardwareInterface>
-      </joint>
-    </transmission>
-    <transmission name="trans_x">
-      <type>transmission_interface/SimpleTransmission</type>
-      <actuator name="$omni_y_motor">
-        <mechanicalReduction>1</mechanicalReduction>
-      </actuator>
-      <joint name="omni_joint_y">
-        <hardwareInterface>hardware_interface/PositionJointInterface</hardwareInterface>
-      </joint>
-    </transmission>
-    <transmission name="trans_y">
-      <type>transmission_interface/SimpleTransmission</type>
-      <actuator name="$omni_x_motor">
-        <mechanicalReduction>1</mechanicalReduction>
-      </actuator>
-      <joint name="omni_joint_x">
-        <hardwareInterface>hardware_interface/PositionJointInterface</hardwareInterface>
-      </joint>
-    </transmission>
-    <gazebo reference="omnitorso_x">
-      <turnGravityOff>false</turnGravityOff>
-      <selfCollide>true</selfCollide>
-    </gazebo>
-    <gazebo reference="omnitorso_y">
-      <turnGravityOff>false</turnGravityOff>
-      <selfCollide>true</selfCollide>
-    </gazebo> -->
-<!--     <gazebo>
-      <plugin name="omnivelma" filename="libomnivelma.so"/>
-    </gazebo> -->
     <gazebo>
       <plugin name="gazebo_ros_force_based_move" filename="libgazebo_ros_force_based_move.so">
@@ -137,97 +31,9 @@
         <y_velocity_i_gain>500.0</y_velocity_i_gain>
         <y_velocity_d_gain>20.0</y_velocity_d_gain>
-        <yaw_velocity_p_gain>600.0</yaw_velocity_p_gain>
-        <yaw_velocity_i_gain>4.0</yaw_velocity_i_gain>
-        <yaw_velocity_d_gain>10.0</yaw_velocity_d_gain>
+        <yaw_velocity_p_gain>300.0</yaw_velocity_p_gain>
+        <yaw_velocity_i_gain>3.0</yaw_velocity_i_gain>
+        <yaw_velocity_d_gain>3.0</yaw_velocity_d_gain>
       </plugin>
     </gazebo>
-<!--             <x_velocity_p_gain>140000.0</x_velocity_p_gain>
-        <x_velocity_i_gain>10000.0</x_velocity_i_gain>
-        <x_velocity_d_gain>10.0</x_velocity_d_gain>
-        <y_velocity_p_gain>140000.0</y_velocity_p_gain>
-        <y_velocity_i_gain>10000.0</y_velocity_i_gain>
-        <y_velocity_d_gain>10.0</y_velocity_d_gain>
-        <yaw_velocity_p_gain>6000.0</yaw_velocity_p_gain>
-        <yaw_velocity_i_gain>20.0</yaw_velocity_i_gain>
-        <yaw_velocity_d_gain>1.0</yaw_velocity_d_gain> -->
-<!--     <link name="omnitorso_y">
-      <inertial>
-        <mass value="20.0"/>
-        <inertia ixx="0" ixy="0" ixz="0" iyy="0" iyz="0" izz="0"/>
-      </inertial>
-      <collision>
-        <origin xyz="0 0 0" rpy="0.0 0 0" />
-        <geometry>
-          <box size="1.0 1.0 0.01" />
-        </geometry>
-        <material name="torso_base">
-          <color rgba="0.3 0.3 0.15 1"/>
-        </material>
-      </collision>
-      <visual>
-        <origin xyz="0 0 0" rpy="0.0 0 0" />
-        <geometry>
-          <box size="1.0 1.0 0.01" />
-        </geometry>
-        <material name="torso_base">
-          <color rgba="0.3 0.3 0.15 1"/>
-        </material>
-      </visual>
-    </link>
-    <link name="omnitorso_x">
-      <inertial>
-        <mass value="20.0"/>
-        <inertia ixx="0" ixy="0" ixz="0" iyy="0" iyz="0" izz="0"/>
-      </inertial>
-      <collision>
-        <origin xyz="0 0 0" rpy="0.0 0 0" />
-        <geometry>
-          <box size="1.0 1.0 0.01" />
-        </geometry>
-        <material name="torso_base">
-          <color rgba="0.3 0.3 0.15 1"/>
-        </material>
-      </collision>
-      <visual>
-        <origin xyz="0 0 0" rpy="0.0 0 0" />
-        <geometry>
-          <box size="1.0 1.0 0.01" />
-        </geometry>
-        <material name="torso_base">
-          <color rgba="0.3 0.3 0.15 1"/>
-        </material>
-      </visual>
-    </link>
-    <joint name="torso_base_joint" type="revolute">
-      <xacro:insert_block name="origin" />
-      <limit lower="-2.0" upper="2.0" effort="100" velocity="1"/>
-      <axis xyz="0 0 1"/>
-      <parent link="${parent}"/>
-      <child link="omnitorso_x"/>
-    </joint>
-    <joint name="omni_joint_y" type="prismatic">
-      <origin xyz="0 0 0" rpy="0 0 0" />
-      <limit lower="-2.0" upper="2.0" effort="100" velocity="1"/>
-      <axis xyz="0 1 0"/>
-      <dynamics damping="10.0"/>
-      <parent link="omnitorso_x"/>
-      <child link="omnitorso_y"/>
-    </joint>
-    <joint name="omni_joint_x" type="prismatic">
-      <origin xyz="0 0 0" rpy="0 0 0" />
-      <limit lower="-2.0" upper="2.0" effort="1000" velocity="1"/>
-      <axis xyz="1 0 0"/>
-      <dynamics damping="10.0"/>
-      <parent link="omnitorso_y"/>
-      <child link="torso_base"/>
-    </joint>
-    <gazebo reference="omnitorso_x">
-      <turnGravityOff>false</turnGravityOff>
-      <selfCollide>true</selfCollide>
-    </gazebo>
-    <gazebo reference="omnitorso_y">
-      <turnGravityOff>false</turnGravityOff>
-      <selfCollide>true</selfCollide>
-    </gazebo> -->
     <joint name="torso_base_joint" type="planar">
       <origin xyz="0 0 0" rpy="0 0 0" />
@@ -268,5 +74,4 @@
       <inertial>
         <mass value="60.0"/>
-        <!-- <mass value="20.0"/> -->
         <inertia ixx="2.94" ixy="0" ixz="0" iyy="2.72" iyz="0" izz="5.40"/>
       </inertial>
@@ -442,5 +247,4 @@
         <mass value="1.6" />
         <wheel_inertia m="1.6" r="0.1016" h="0.05" />
-        <!-- <inertia ixx="0.004738485" ixy="0" ixz="0" iyy="0.008" iyz="0" izz="0.004738485" /> -->
       </inertial>
       <visual name="wheel_fl_middle">
@@ -492,5 +296,4 @@
       <visual>
         <origin xyz="0 0 0.52" rpy="0 0 0"/>
-        <!-- <origin xyz="0 0 0.364" rpy="0 0 0"/> -->
         <geometry>
           <mesh filename="package://velma_description/meshes/collision/torso0_collision.stl" />
@@ -502,5 +305,4 @@
       <collision>
         <origin xyz="0 0 0.52" rpy="0 0 0"/>
-        <!-- <origin xyz="0 0 0.364" rpy="0 0 0"/> -->
         <geometry>
           <mesh filename="package://velma_description/meshes/collision/torso0_collision.stl" />

Commit message: cleanup trash

File: velma_description/defs/monokl.urdf.xacro (robot description, xacro)
@@ -64,5 +64,5 @@
       <sensor type="gpu_ray" name="${name}">
       <pose>0 0 0 0 0 0</pose>
-      <visualize>false</visualize>
+      <visualize>true</visualize>
       <update_rate>40</update_rate>
       <ray>

File: velma_description/defs/torso.urdf.xacro (robot description, xacro)
@@ -34,4 +34,5 @@
         <yaw_velocity_i_gain>3.0</yaw_velocity_i_gain>
         <yaw_velocity_d_gain>3.0</yaw_velocity_d_gain>
+        <useRealOdom>true</useRealOdom>
       </plugin>
     </gazebo>
@@ -61,13 +62,8 @@
       </visual>
       <collision>
-        <origin xyz="-0.081 0 0.1225" rpy="0.0 0 0" />
-        <geometry>
-          <mesh filename="package://omnivelma/meshes/collider/base.dae" />
-        </geometry>
-      </collision>
-      <collision>
-        <origin xyz="-0.035 0 0.25" rpy="0.0 0 0" />
-        <geometry>
-          <box size="0.364 0.32 0.15" />
+        <origin xyz="0.01 0 0.1225" rpy="0.0 0 0" />
+        <geometry>
+          <box size="0.907 0.75 0.15" />
+          <!-- <mesh filename="package://omnivelma/meshes/collider/base.dae" /> -->
         </geometry>
       </collision>
@@ -108,10 +104,4 @@
         </geometry>
       </visual>
-      <collision>
-        <origin xyz="0.364 0 0.1225" rpy="0 0 0"/>
-        <geometry>
-          <mesh filename="package://omnivelma/meshes/collider/front.dae" />
-        </geometry>
-      </collision>
       <inertial>
         <mass value="15.0"/>
@@ -247,4 +237,5 @@
         <mass value="1.6" />
         <wheel_inertia m="1.6" r="0.1016" h="0.05" />
+        <!-- <inertia ixx="0.004738485" ixy="0" ixz="0" iyy="0.008" iyz="0" izz="0.004738485" /> -->
       </inertial>
       <visual name="wheel_fl_middle">
@@ -315,11 +306,11 @@
         </geometry>
       </self_collision_checking>
-<!--       <self_collision_checking>
+<!--
+      <self_collision_checking>
         <origin xyz="-0.1 0.0 0.45" rpy="0 0 0"/>
         <geometry>
           <capsule radius="0.18" length="0.4"/>
         </geometry>
-      </self_collision_checking>
- -->
+      </self_collision_checking> -->
       <inertial>
         <mass value="30.0"/>

Commit message: added use_gpu arg

File: velma_description/defs/monokl.urdf.xacro (robot description, xacro)
@@ -4,4 +4,11 @@
                         xmlns:sensor="http://playerstage.sourceforge.net/gazebo/xmlschema/#sensor"
                         xmlns:xacro="http://www.ros.org/wiki/xacro">
+  <xacro:arg name="use_gpu" default="true"/>
+  <xacro:if value="$(arg use_gpu)">
+    <xacro:property name="gpu_prefix" value="gpu_" />
+  </xacro:if>
+  <xacro:unless value="$(arg use_gpu)">
+    <xacro:property name="gpu_prefix" value="" />
+  </xacro:unless>
   <xacro:macro name="monokl" params="parent name *origin">
   	<joint name="${name}_joint" type="fixed">
@@ -62,8 +69,11 @@
     <gazebo reference="${name}_heart">
       <selfCollide>true</selfCollide>
-      <sensor type="gpu_ray" name="${name}">
+      <sensor type="${gpu_prefix}ray" name="${name}">
       <pose>0 0 0 0 0 0</pose>
       <visualize>true</visualize>
       <update_rate>40</update_rate>
+      <xacro:unless value="$(arg use_gpu)">
+        <always_on>true</always_on>
+      </xacro:unless>
       <ray>
         <scan>
@@ -90,5 +100,5 @@
         </noise>
       </ray>
-      <plugin name="gazebo_ros_head_hokuyo_controller" filename="libgazebo_ros_gpu_laser.so">
+      <plugin name="gazebo_ros_head_hokuyo_controller" filename="libgazebo_ros_${gpu_prefix}laser.so">
         <topicName>/${name}/scan</topicName>
         <frameName>${name}_heart</frameName>

Commit message: mobile base

File: velma_description/defs/monokl.urdf.xacro (robot description, xacro)
@@ -30,10 +30,10 @@
       	</geometry>
       </visual>
-      <collision>
+      <!--<collision>
         <origin xyz="0 0 0" rpy="0 0 0"/>
         <geometry>
           <cylinder radius="0.051" length="0.131" />
         </geometry>
-      </collision>
+      </collision>-->
       <inertial>
         <mass value="1.1"/>
@@ -52,10 +52,10 @@
           </geometry>
         </visual>
-        <collision>
+        <!--<collision>
           <origin xyz="0 0 0" rpy="0 0 0"/>
           <geometry>
             <cylinder radius="0.04" length="0.04" />
           </geometry>
-        </collision>
+        </collision>-->
     </link>
     <joint name="${name}_heart_fix" type="fixed">

File: velma_description/defs/torso.urdf.xacro (robot description, xacro)
@@ -96,33 +96,4 @@
     </joint>
     <link name="torso_link0">
-<!--
-      <visual>
-        <origin xyz="0 0 0.219" rpy="0.0 0 0" />
-        <geometry>
-          <mesh filename="package://velma_description/meshes/base_asm.STL" />
-        </geometry>
-        <material name="torso_base">
-          <color rgba="0.5 0.5 0.5 1"/>
-        </material>
-      </visual>
-      <visual>
-        <origin xyz="-0.01 0 0.93" rpy="0.0 0 0" />
-        <geometry>
-          <box size="0.28 0.24 0.32" />
-        </geometry>
-        <material name="torso_base">
-          <color rgba="0.5 0.5 0.5 1"/>
-        </material>
-      </visual>
-      <visual>
-        <origin xyz="0 0.0 1.055" rpy="0 0 0.0" />
-        <geometry>
-          <mesh filename="package://velma_description/meshes/top_base_asm.STL" />
-        </geometry>
-        <material name="torso_asm">
-          <color rgba="1.0 0.487 0 1.0"/>
-        </material>
-      </visual>
--->
       <visual>
         <origin xyz="0 0 0.52" rpy="0 0 0"/>

File: velma_description/defs/torso_mobile.urdf.xacro (robot description, xacro)
@@ -290,5 +290,5 @@
         <origin xyz="0 0 0.52" rpy="0 0 0"/>
         <geometry>
-          <mesh filename="package://velma_description/meshes/collision/torso0_mobile_collision.stl" />
+          <mesh filename="package://velma_description/meshes/collision/torso0_collision.stl" />
         </geometry>
         <material name="torso_base">
@@ -296,10 +296,32 @@
         </material>
       </visual>
-      <collision>
-        <origin xyz="0 0 0.52" rpy="0 0 0"/>
-        <geometry>
-          <mesh filename="package://velma_description/meshes/collision/torso0_mobile_collision.stl" />
-        </geometry>
-      </collision>
+      <xacro:if value="${collision_detector == 'fcl'}">
+        <collision>
+          <origin xyz="0 0 0.52" rpy="0 0 0"/>
+          <geometry>
+            <mesh filename="package://velma_description/meshes/collision/torso0_mobile_collision.stl" />
+          </geometry>
+        </collision>
+      </xacro:if>
+      <xacro:if value="${collision_detector == 'dart'}">
+        <collision>
+          <origin xyz="0 0 0.968570022583" rpy="0 0 0"/>
+          <geometry>
+            <box size="0.30822044611 0.276354163885 0.45334654808"/>
+          </geometry>
+        </collision>
+        <collision>
+          <origin xyz="0 0 1.18425571918" rpy="${M_PI/4} 0 0"/>
+          <geometry>
+            <box size="0.316696882248 0.19 0.19"/>
+          </geometry>
+        </collision>
+        <collision>
+          <origin xyz="-0.0265109799802 0 0.505967736244" rpy="0 0 0"/>
+          <geometry>
+            <box size="0.353161275387 0.255815982819 0.5"/>
+          </geometry>
+        </collision>
+      </xacro:if>
       <self_collision_checking>
         <origin xyz="0 0.0 0.8" rpy="0 0 0"/>
@@ -323,4 +345,5 @@
       <turnGravityOff>false</turnGravityOff>
       <selfCollide>true</selfCollide>
+      <material>Gazebo/DarkGrey</material>
     </gazebo>
   </xacro:macro>
