Commit message: fix.

File: velma_description/defs/head.urdf.xacro (robot description, xacro)
@@ -1,26 +1,59 @@
 <?xml version="1.0"?>
 <robot>
-  <include filename="$(find velma_description)/defs/camera.urdf.xacro" />
   <macro name="velma_head" params="parent *origin">
-    <joint name="head_frame_joint" type="fixed">
+    <joint name="head_base_joint" type="fixed">
       <insert_block name="origin" />
       <parent link="${parent}"/>
-      <child link="head_frame"/>
+      <child link="head_base"/>
     </joint>
-    <link name="head_frame">
+    <link name="head_base">
+       <visual>
+        <origin xyz="0 0 0.0" rpy="0 0 0" />
+        <geometry>
+          <mesh filename="package://velma_description/meshes/head_base.STL" />
+        </geometry>
+        <material name="torso_gray">
+          <color rgba="0.5 0.5 0.5 1"/>
+        </material>
+      </visual>
+    </link>
+    <joint name="head_pan_motor_joint" type="fixed">
+      <origin xyz="0 0 0.025" rpy="0 0 0" />
+      <parent link="head_base"/>
+      <child link="head_pan_motor"/>
+    </joint>
+    <link name="head_pan_motor">
+       <visual>
+        <origin xyz="0 0 0" rpy="0 0 0" />
+        <geometry>
+          <mesh filename="package://velma_description/meshes/head_pan.STL" />
+        </geometry>
+        <material name="torso_gray">
+          <color rgba="0.5 0.5 0.5 1"/>
+        </material>
+      </visual>
     </link>
     <!-- pan -->
     <joint name="head_pan_joint" type="revolute">
-      <origin xyz="0 0 0" rpy="0 0 0"/>
+      <origin xyz="0 0 0.062" rpy="0 0 0"/>
       <axis xyz="0 0 1"/>
-      <parent link="head_frame"/>
+      <parent link="head_pan_motor"/>
       <child link="head_pan_link"/>
-      <limit lower="-1.57" upper="1.57" effort="100" velocity="100"/>
+      <limit lower="-1.57" upper="1.57" effort="100" velocity="1.57"/>
     </joint>
     <link name="head_pan_link">
+      <visual>
+        <origin xyz="0 0 0" rpy="0 0 0" />
+        <geometry>
+          <mesh filename="package://velma_description/meshes/head_tilt.STL" />
+        </geometry>
+        <material name="torso_gray">
+          <color rgba="0.5 0.5 0.5 1"/>
+        </material>
+      </visual>
     </link>
     <!-- tilt -->
     <joint name="head_tilt_joint" type="revolute">
-      <origin xyz="0 0 0.0" rpy="-1.57 0.0 0" />
+      <origin xyz="0 0 0.048" rpy="1.57 0.0 0" />
       <axis xyz="0 0 1"/>
       <parent link="head_pan_link"/>
@@ -28,5 +61,15 @@
       <limit lower="-1.57" upper="1.57" effort="100" velocity="100"/>
     </joint>
-    <link name="head_tilt_link"/>
+    <link name="head_tilt_link">
+      <visual>
+        <origin xyz="0 0 0.04219" rpy="0 0 0" />
+        <geometry>
+          <mesh filename="package://velma_description/meshes/head_top.STL" />
+        </geometry>
+        <material name="torso_gray">
+          <color rgba="0.5 0.5 0.5 1"/>
+        </material>
+      </visual>
+    </link>
     <!-- sensors -->
     <head_camera parent="head_tilt_link" name="stereo_left">

File: velma_description/robots/velma.urdf.xacro (robot description, xacro)
@@ -6,4 +6,6 @@
 	 name="velma">
   <xacro:include filename="$(find velma_description)/calibration/default_cal.xml"/>
+  <xacro:include filename="$(find velma_description)/defs/torso.urdf.xacro"/>
+  <xacro:include filename="$(find velma_description)/defs/head.urdf.xacro" />
   <xacro:include filename="$(find lwr_defs)/defs/kuka_lwr_arm_defs.xml"/>
   <xacro:include filename="$(find lwr_defs)/defs/materials.xml"/>
@@ -11,49 +13,10 @@
 <!--
   <include filename="$(find velma_defs)/defs/kinect_camera.urdf.xacro" />
-  <include filename="$(find velma_defs)/defs/head.urdf.xacro" /> -->
+   -->
   <property name="M_PI" value="3.1415926535897931" />
   <link name="world" />
-  <joint name="arm_world_joint" type="fixed">
+  <velma_torso parent="world" >
     <origin xyz="0 0 0.1" rpy="0 0 0"/>
-    <parent link="world"/>
-    <child link="torso_base"/>
-  </joint>
-  <link name="torso_base">
-  </link>
-  <joint name="torso_0_joint" type="revolute">
-    <origin xyz="0 0 0.0" rpy="0 0 0"/>
-    <axis xyz="0 0 1"/>
-    <limit lower="-1.57" upper="1.57" effort="100" velocity="100"/>
-    <parent link="torso_base"/>
-    <child link="torso_link0"/>
-  </joint>
-  <link name="torso_link0">
-  </link>
-  <joint name="torso_1_joint" type="revolute">
-    <origin xyz="0 0 0.80" rpy="${M_PI/2} 0 0"/>
-    <axis xyz="0 0 -1"/>
-    <limit lower="${M_PI/4}" upper="${105 * M_PI/180}" effort="100" velocity="100"/>
-    <parent link="torso_link0"/>
-    <child link="torso_link1"/>
-  </joint>
-  <link name="torso_link1">
-  </link>
-  <joint name="torso_2_joint" type="revolute">
-    <origin xyz="0.375 0 0" rpy="0 0 0"/>
-    <axis xyz="0 0 -1"/>
-    <limit lower="-1.57" upper="1.57" effort="100" velocity="100"/>
-    <mimic joint="torso_1_joint" multiplier="-1"/>
-    <parent link="torso_link1"/>
-    <child link="torso_link2"/>
-  </joint>
-  <link name="torso_link2">
-    <visual>
-      <origin xyz="0 0.04 0" rpy="${-M_PI/2.0} 0 0.0" />
-      <!--origin xyz="-0.03 -0.07 0" rpy="0 0 -1.57"-->
-      <geometry>
-        <mesh filename="package://velma_description/meshes/arm_base.STL" />
-      </geometry>
-    </visual>
-  </link>
+  </velma_torso>
   <kuka_lwr_arm parent="torso_link2" name="right" right="1">
     <origin xyz="0 0.1641 0.07943" rpy="${-M_PI/6} 0 0"/>
@@ -73,4 +36,5 @@
         <mesh filename="package://velma_description/meshes/gripper_mount.STL" />
       </geometry>
+      <material name="Orange"/>
     </visual>
   </link>
@@ -86,4 +50,5 @@
         <mesh filename="package://velma_description/meshes/gripper_mount.STL" />
       </geometry>
+      <material name="Orange"/>
     </visual>
   </link>
@@ -94,3 +59,6 @@
     <origin xyz="-0.115 0.0 -0.078" rpy="0 ${-M_PI/2} 0"/>
   </xacro:barret_hand>
+  <velma_head parent="torso_link2">
+    <origin xyz="0 0.253 0.0" rpy="${-M_PI/2} 0 0"/>
+  </velma_head>
 </robot>

Commit message: collision model

File: velma_description/defs/head.urdf.xacro (robot description, xacro)
@@ -33,4 +33,10 @@
         </material>
       </visual>
+      <self_collision_checking>
+        <origin xyz="0.0 0 0.04" rpy="0 0 0"/>
+        <geometry>
+          <capsule radius="0.07" length="0.08"/>
+        </geometry>
+      </self_collision_checking>
     </link>
     <!-- pan -->
@@ -71,4 +77,16 @@
         </material>
       </visual>
+      <self_collision_checking>
+        <origin xyz="0.0 0.12 0.0" rpy="-1.57075 0 0"/>
+        <geometry>
+          <capsule radius="0.07" length="0.24"/>
+        </geometry>
+      </self_collision_checking>
+      <self_collision_checking>
+        <origin xyz="0.05 0.18 0.0" rpy="0 0 0"/>
+        <geometry>
+          <capsule radius="0.07" length="0.23"/>
+        </geometry>
+      </self_collision_checking>
     </link>
     <!-- sensors -->

File: velma_description/defs/torso.urdf.xacro (robot description, xacro)
@@ -26,4 +26,10 @@
         </material>
       </visual>
+      <self_collision_checking>
+        <origin xyz="-0.2 0.0 0.6" rpy="1.57075 0 0"/>
+        <geometry>
+          <capsule radius="0.20" length="0.9"/>
+        </geometry>
+      </self_collision_checking>
     </link>
     <joint name="torso_0_joint" type="revolute">

File: velma_description/robots/velma.urdf.xacro (robot description, xacro)
@@ -38,4 +38,10 @@
       <material name="Orange"/>
     </visual>
+    <self_collision_checking>
+      <origin xyz="0.05 0.0 -0.03" rpy="0 -0.81 0"/>
+      <geometry>
+        <capsule radius="0.055" length="0.14"/>
+      </geometry>
+    </self_collision_checking>
   </link>
   <joint name="left_gripper_mount_joint" type="fixed">
@@ -52,4 +58,10 @@
       <material name="Orange"/>
     </visual>
+    <self_collision_checking>
+      <origin xyz="0.05 0.0 -0.03" rpy="0 -0.81 0"/>
+      <geometry>
+        <capsule radius="0.055" length="0.14"/>
+      </geometry>
+    </self_collision_checking>
   </link>
   <xacro:barret_hand prefix="right" parent="right_arm_7_link">

Commit message: Add new head to URDF.

File: velma_description/defs/head.urdf.xacro (robot description, xacro)
@@ -1,4 +1,8 @@
 <?xml version="1.0"?>
-<robot>
+<robot xmlns:controller="http://playerstage.sourceforge.net/gazebo/xmlschema/#controller"
+                        xmlns:interface="http://playerstage.sourceforge.net/gazebo/xmlschema/#interface"
+                        xmlns:sensor="http://playerstage.sourceforge.net/gazebo/xmlschema/#sensor"
+                        xmlns:xacro="http://playerstage.sourceforge.net/gazebo/xmlschema/#interface">
+  <xacro:include filename="$(find velma_description)/defs/camera.urdf.xacro" />
   <macro name="velma_head" params="parent *origin">
     <joint name="head_base_joint" type="fixed">
@@ -56,5 +60,5 @@
     <joint name="head_tilt_joint" type="revolute">
       <origin xyz="0 0 0.048" rpy="1.57 0.0 0" />
-      <axis xyz="0 0 1"/>
+      <axis xyz="0 0 -1"/>
       <parent link="head_pan_link"/>
       <child link="head_tilt_link"/>
@@ -74,6 +78,4 @@
     <!-- sensors -->
     <head_camera parent="head_tilt_link" name="stereo_left">
-      <!--<origin xyz="0.074819 -0.19424 0.039144" rpy="1.572 -0.0046408 0.0147"/> -->
-      <!-- <origin xyz="0.072474    -0.21002    0.043726" rpy="1.5767  -0.0094749   0.0058925"/> -->
       <origin xyz="${cal_head_to_stereo_left_x} ${cal_head_to_stereo_left_y} ${cal_head_to_stereo_left_z}"
               rpy="${cal_head_to_stereo_left_roll} ${cal_head_to_stereo_left_pitch} ${cal_head_to_stereo_left_yaw}"/>
@@ -82,22 +84,4 @@
       <origin xyz="0.0 -0.09 0.0" rpy="0 0 0"/>
     </head_camera>
-    <head_camera parent="head_tilt_link" name="kinect_left_rgb">
-      <!--<origin xyz="0.013309 -0.010124 -0.06841" rpy="1.5634 -0.022662 0.37293"/> -->
-      <!--<origin xyz="0.019408   -0.010485   -0.088064" rpy="1.5637  -0.0097296     0.36447"/>-->
-      <origin xyz="${cal_stereo_left_to_kinect_left_x} ${cal_stereo_left_to_kinect_left_y} ${cal_stereo_left_to_kinect_left_z}"
-              rpy="${cal_stereo_left_to_kinect_left_roll} ${cal_stereo_left_to_kinect_left_pitch} ${cal_stereo_left_to_kinect_left_yaw}"/>
-    </head_camera>
-    <head_camera parent="kinect_left_rgb_link" name="kinect_left_ir">
-      <origin xyz="0.0 0.03 0.0" rpy="0 0 0"/>
-    </head_camera>
-    <head_camera parent="head_tilt_link" name="kinect_right_rgb">
-      <!--<origin xyz="0.00045739 -0.071104 -0.074766" rpy="1.5892 -0.035955 -0.34978"/> -->
-      <!--<origin xyz="-0.034936    -0.05614   -0.084153" rpy="1.588   -0.024981    -0.37211"/>-->
-      <origin xyz="${cal_stereo_left_to_kinect_right_x} ${cal_stereo_left_to_kinect_right_y} ${cal_stereo_left_to_kinect_right_z}"
-              rpy="${cal_stereo_left_to_kinect_right_roll} ${cal_stereo_left_to_kinect_right_pitch} ${cal_stereo_left_to_kinect_right_yaw}"/>
-    </head_camera>
-    <head_camera parent="kinect_right_rgb_link" name="kinect_right_ir">
-      <origin xyz="0.0 0.03 0.0" rpy="0 0 0"/>
-    </head_camera>
   </macro>
 </robot>

File: velma_description/robots/velma.urdf.xacro (robot description, xacro)
@@ -56,7 +56,21 @@
     <origin xyz="0.115 0.0 -0.078" rpy="0 ${M_PI/2} 0"/>
   </xacro:barret_hand>
+  <joint name="right_gripper_calib_joint" type="fixed">
+    <origin xyz="0 0.0445 0.031" rpy="0 0 0"/>
+    <parent link="right_HandPalmLink"/>
+    <child link="right_gripper_calib_link"/>
+  </joint>
+  <link name="right_gripper_calib_link">
+  </link>
   <xacro:barret_hand prefix="left" parent="left_arm_7_link">
     <origin xyz="-0.115 0.0 -0.078" rpy="0 ${-M_PI/2} 0"/>
   </xacro:barret_hand>
+  <joint name="left_gripper_calib_joint" type="fixed">
+    <origin xyz="0 0.0445 0.031" rpy="0 0 0"/>
+    <parent link="left_HandPalmLink"/>
+    <child link="left_gripper_calib_link"/>
+  </joint>
+  <link name="left_gripper_calib_link">
+  </link>
   <velma_head parent="torso_link2">
     <origin xyz="0 0.253 0.0" rpy="${-M_PI/2} 0 0"/>

Commit message: add calibration data.

File: velma_description/defs/head.urdf.xacro (robot description, xacro)
@@ -96,10 +96,14 @@
     <!-- sensors -->
     <head_camera parent="head_tilt_link" name="stereo_left">
-      <origin xyz="${cal_head_to_stereo_left_x} ${cal_head_to_stereo_left_y} ${cal_head_to_stereo_left_z}"
-              rpy="${cal_head_to_stereo_left_roll} ${cal_head_to_stereo_left_pitch} ${cal_head_to_stereo_left_yaw}"/>
+      <origin xyz="${cal_stereo_left_joint_x} ${cal_stereo_left_joint_y} ${cal_stereo_left_joint_z}"
+              rpy="${cal_stereo_left_joint_roll} ${cal_stereo_left_joint_pitch} ${cal_stereo_left_joint_yaw}"/>
     </head_camera>
     <head_camera parent="stereo_left_link" name="stereo_right">
       <origin xyz="0.0 -0.09 0.0" rpy="0 0 0"/>
     </head_camera>
+    <head_camera parent="head_tilt_link" name="head_kinect_rgb">
+      <origin xyz="${cal_head_kinect_rgb_joint_x} ${cal_head_kinect_rgb_joint_y} ${cal_head_kinect_rgb_joint_z}"
+              rpy="${cal_head_kinect_rgb_joint_roll} ${cal_head_kinect_rgb_joint_pitch} ${cal_head_kinect_rgb_joint_yaw}"/>
+    </head_camera>
   </macro>
 </robot>

File: velma_description/robots/velma.urdf.xacro (robot description, xacro)
@@ -23,5 +23,5 @@
   </kuka_lwr_arm>
   <kuka_lwr_arm parent="torso_link2" name="left" right="1">
-    <origin xyz="0 0.1641 -0.07943" rpy="${-5*M_PI/6} 0 0"/>
+    <origin xyz="${cal_torso_link2_left_arm_base_joint_x} ${cal_torso_link2_left_arm_base_joint_y} ${cal_torso_link2_left_arm_base_joint_z}" rpy="${cal_torso_link2_left_arm_base_joint_roll} ${cal_torso_link2_left_arm_base_joint_pitch} ${cal_torso_link2_left_arm_base_joint_yaw}"/>
   </kuka_lwr_arm>
   <joint name="right_gripper_mount_joint" type="fixed">
@@ -69,6 +69,6 @@
   </xacro:barret_hand>
   <joint name="right_gripper_calib_joint" type="fixed">
-    <origin xyz="0 0.0445 0.031" rpy="0 0 0"/>
-    <parent link="right_HandPalmLink"/>
+    <origin xyz="${cal_right_gripper_calib_link_x} ${cal_right_gripper_calib_link_y} ${cal_right_gripper_calib_link_z}" rpy="0 0 0"/>
+    <parent link="right_arm_7_link"/>
     <child link="right_gripper_calib_link"/>
   </joint>
@@ -79,12 +79,16 @@
   </xacro:barret_hand>
   <joint name="left_gripper_calib_joint" type="fixed">
-    <origin xyz="0 0.0445 0.031" rpy="0 0 0"/>
-    <parent link="left_HandPalmLink"/>
+    <origin xyz="${cal_left_gripper_calib_link_x} ${cal_left_gripper_calib_link_y} ${cal_left_gripper_calib_link_z}" rpy="0 0 0"/>
+    <parent link="left_arm_7_link"/>
     <child link="left_gripper_calib_link"/>
   </joint>
   <link name="left_gripper_calib_link">
   </link>
+  <head_camera parent="left_arm_7_link" name="left_hand_camera">
+      <origin xyz="${cal_left_hand_camera_joint_x} ${cal_left_hand_camera_joint_y} ${cal_left_hand_camera_joint_z}"
+              rpy="${cal_left_hand_camera_joint_roll} ${cal_left_hand_camera_joint_pitch} ${cal_left_hand_camera_joint_yaw}"/>
+  </head_camera>
   <velma_head parent="torso_link2">
-    <origin xyz="0 0.253 0.0" rpy="${-M_PI/2} 0 0"/>
+    <origin xyz="${cal_head_base_joint_x} ${cal_head_base_joint_y} ${cal_head_base_joint_z}" rpy="${cal_head_base_joint_roll} ${cal_head_base_joint_pitch} ${cal_head_base_joint_yaw}"/>
   </velma_head>
 </robot>

Commit message: add cameras calibration to repo.

File: velma_description/defs/head.urdf.xacro (robot description, xacro)
@@ -100,5 +100,6 @@
     </head_camera>
     <head_camera parent="stereo_left_link" name="stereo_right">
-      <origin xyz="0.0 -0.09 0.0" rpy="0 0 0"/>
+      <origin xyz="${cal_stereo_right_joint_x} ${cal_stereo_right_joint_y} ${cal_stereo_right_joint_z}"
+              rpy="${cal_stereo_right_joint_roll} ${cal_stereo_right_joint_pitch} ${cal_stereo_right_joint_yaw}"/>
     </head_camera>
     <head_camera parent="head_tilt_link" name="head_kinect_rgb">
