Commit message: added collision geoms to urdf of Velma

File: velma_description/defs/head.urdf.xacro (robot description, xacro)
@@ -21,4 +21,10 @@
         </material>
       </visual>
+      <collision>
+        <origin xyz="0 0 0.0" rpy="0 0 0" />
+        <geometry>
+          <mesh filename="package://velma_description/meshes/collision/head_base_collision.STL" />
+        </geometry>
+      </collision>
     </link>
     <joint name="head_pan_motor_joint" type="fixed">
@@ -37,4 +43,10 @@
         </material>
       </visual>
+      <collision>
+        <origin xyz="0 0 0.0308" rpy="0 0 0" />
+        <geometry>
+          <box size="0.14 0.09 0.06" />
+        </geometry>
+      </collision>
       <self_collision_checking>
         <origin xyz="0.0 0 0.04" rpy="0 0 0"/>
@@ -62,4 +74,10 @@
         </material>
       </visual>
+      <collision>
+        <origin xyz="0 -0.00921 0.04463" rpy="0 0 0" />
+        <geometry>
+          <box size="0.08 0.08 0.08" />
+        </geometry>
+      </collision>
     </link>
     <!-- tilt -->
@@ -81,4 +99,10 @@
         </material>
       </visual>
+      <collision>
+        <origin xyz="0 0 0.04219" rpy="0 0 0 " />
+        <geometry>
+          <mesh filename="package://velma_description/meshes/collision/head_top_collision.STL" />
+        </geometry>
+      </collision>
       <self_collision_checking>
         <origin xyz="0.0 0.12 0.0" rpy="-1.57075 0 0"/>

File: velma_description/defs/torso.urdf.xacro (robot description, xacro)
@@ -9,16 +9,7 @@
     <link name="torso_base">
       <visual>
-        <origin xyz="0 0 0.05" rpy="0.0 0 0" />
+        <origin xyz="0 0 0" rpy="0.0 0 0" />
         <geometry>
-          <box size="0.7 0.82 0.1" />
-        </geometry>
-        <material name="torso_base">
-          <color rgba="0.1 0.1 0.1 1"/>
-        </material>
-      </visual>
-      <visual>
-        <origin xyz="0 0 0.16" rpy="0.0 0 0" />
-        <geometry>
-          <box size="0.41 0.41 0.12" />
+          <mesh filename="package://velma_description/meshes/torso_base.STL" />
         </geometry>
         <material name="torso_base">
@@ -50,4 +41,10 @@
         </material>
       </visual>
+      <collision>
+        <origin xyz="-0.03338 0 0.519" rpy="0 0 0"/>
+        <geometry>
+          <box size="0.34 0.3 0.6"/>
+        </geometry>
+      </collision>
       <self_collision_checking>
         <origin xyz="0 0.0 0.4" rpy="0 0 0"/>
@@ -101,4 +98,10 @@
         </material>
       </visual>
+      <collision>
+        <origin xyz="0 0 -0.09875" rpy="${-M_PI/2} 0 ${-M_PI/2}" />
+        <geometry>
+          <mesh filename="package://velma_description/meshes/collision/connector2_collision.STL" />
+        </geometry>
+      </collision>
     </link>
     <joint name="torso_1_joint_viz2" type="revolute">
@@ -120,4 +123,10 @@
         </material>
       </visual>
+      <collision>
+        <origin xyz="0 0 -0.09875" rpy="${-M_PI/2} 0 ${-M_PI/2}" />
+        <geometry>
+          <mesh filename="package://velma_description/meshes/collision/connector_collision.STL" />
+        </geometry>
+      </collision>
     </link>
     <joint name="torso_2_joint" type="revolute">
@@ -137,4 +146,11 @@
         <material name="Orange"/>
       </visual>
+      <collision>
+        <origin xyz="0 0.0 0" rpy="${-M_PI/2.0} 0 0.0" />
+        <geometry>
+          <mesh filename="package://velma_description/meshes/collision/top_base_asm_collision.STL" />
+        </geometry>
+        <material name="Orange"/>
+      </collision>
     </link>
   </macro>

File: velma_description/robots/velma.urdf.xacro (robot description, xacro)
@@ -38,4 +38,10 @@
       <material name="Orange"/>
     </visual>
+    <collision>
+      <origin xyz="0 0 0" rpy="0 0 0"/>
+      <geometry>
+        <mesh filename="package://velma_description/meshes/collision/gripper_mount_collision.STL"/>
+      </geometry>
+    </collision>
     <self_collision_checking>
       <origin xyz="0.05 0.0 -0.03" rpy="0 -0.81 0"/>
@@ -58,4 +64,10 @@
       <material name="Orange"/>
     </visual>
+    <collision>
+      <origin xyz="0 0 0" rpy="0 0 0"/>
+      <geometry>
+        <mesh filename="package://velma_description/meshes/collision/gripper_mount_collision.STL"/>
+      </geometry>
+    </collision>
     <self_collision_checking>
       <origin xyz="0.05 0.0 -0.03" rpy="0 -0.81 0"/>

File: velma_description/robots/velma_export.urdf.xacro (robot description, xacro)
@@ -6,4 +6,6 @@
 	 name="velma">
   <xacro:include filename="$(find velma_description)/calibration/default_cal.xml"/>
+  <xacro:include filename="$(find velma_description)/defs/torso_export.urdf.xacro"/>
+  <xacro:include filename="$(find velma_description)/defs/head_export.urdf.xacro" />
   <xacro:include filename="$(find lwr_defs)/defs/kuka_lwr_arm_defs_export.xml"/>
   <xacro:include filename="$(find lwr_defs)/defs/materials.xml"/>
@@ -11,49 +13,10 @@
 <!--
   <include filename="$(find velma_defs)/defs/kinect_camera.urdf.xacro" />
-  <include filename="$(find velma_defs)/defs/head.urdf.xacro" /> -->
+   -->
   <property name="M_PI" value="3.1415926535897931" />
   <link name="world" />
-  <joint name="arm_world_joint" type="fixed">
+  <velma_torso parent="world" >
     <origin xyz="0 0 0.1" rpy="0 0 0"/>
-    <parent link="world"/>
-    <child link="torso_base"/>
-  </joint>
-  <link name="torso_base">
-  </link>
-  <joint name="torso_0_joint" type="revolute">
-    <origin xyz="0 0 0.0" rpy="0 0 0"/>
-    <axis xyz="0 0 1"/>
-    <limit lower="-1.57" upper="1.57" effort="100" velocity="100"/>
-    <parent link="torso_base"/>
-    <child link="torso_link0"/>
-  </joint>
-  <link name="torso_link0">
-  </link>
-  <joint name="torso_1_joint" type="revolute">
-    <origin xyz="0 0 0.80" rpy="${M_PI/2} 0 0"/>
-    <axis xyz="0 0 -1"/>
-    <limit lower="-${M_PI/2}" upper="${105 * M_PI/180}" effort="100" velocity="100"/>
-    <parent link="torso_link0"/>
-    <child link="torso_link1"/>
-  </joint>
-  <link name="torso_link1">
-  </link>
-  <joint name="torso_2_joint" type="revolute">
-    <origin xyz="0.375 0 0" rpy="0 0 0"/>
-    <axis xyz="0 0 -1"/>
-    <limit lower="-1.57" upper="${M_PI/2}" effort="100" velocity="100"/>
-    <mimic joint="torso_1_joint" multiplier="-1"/>
-    <parent link="torso_link1"/>
-    <child link="torso_link2"/>
-  </joint>
-  <link name="torso_link2">
-    <visual>
-      <origin xyz="0 0.04 0" rpy="${-M_PI/2.0} 0 0.0" />
-      <!--origin xyz="-0.03 -0.07 0" rpy="0 0 -1.57"-->
-      <geometry>
-        <mesh filename="package://velma_description/meshes/arm_base_export.STL" />
-      </geometry>
-    </visual>
-  </link>
+  </velma_torso>
   <kuka_lwr_arm parent="torso_link2" name="right" right="1">
     <origin xyz="0 0.1641 0.07943" rpy="${-M_PI/6} 0 0"/>
@@ -73,5 +36,12 @@
         <mesh filename="package://velma_description/meshes/gripper_mount_export.STL" />
       </geometry>
+      <material name="Orange"/>
     </visual>
+    <self_collision_checking>
+      <origin xyz="0.05 0.0 -0.03" rpy="0 -0.81 0"/>
+      <geometry>
+        <capsule radius="0.055" length="0.14"/>
+      </geometry>
+    </self_collision_checking>
   </link>
   <joint name="left_gripper_mount_joint" type="fixed">
@@ -86,11 +56,35 @@
         <mesh filename="package://velma_description/meshes/gripper_mount_export.STL" />
       </geometry>
+      <material name="Orange"/>
     </visual>
+    <self_collision_checking>
+      <origin xyz="0.05 0.0 -0.03" rpy="0 -0.81 0"/>
+      <geometry>
+        <capsule radius="0.055" length="0.14"/>
+      </geometry>
+    </self_collision_checking>
   </link>
   <xacro:barret_hand prefix="right" parent="right_arm_7_link">
     <origin xyz="0.115 0.0 -0.078" rpy="0 ${M_PI/2} 0"/>
   </xacro:barret_hand>
+  <joint name="right_gripper_calib_joint" type="fixed">
+    <origin xyz="0 0.0445 0.031" rpy="0 0 0"/>
+    <parent link="right_HandPalmLink"/>
+    <child link="right_gripper_calib_link"/>
+  </joint>
+  <link name="right_gripper_calib_link">
+  </link>
   <xacro:barret_hand prefix="left" parent="left_arm_7_link">
     <origin xyz="-0.115 0.0 -0.078" rpy="0 ${-M_PI/2} 0"/>
   </xacro:barret_hand>
+  <joint name="left_gripper_calib_joint" type="fixed">
+    <origin xyz="0 0.0445 0.031" rpy="0 0 0"/>
+    <parent link="left_HandPalmLink"/>
+    <child link="left_gripper_calib_link"/>
+  </joint>
+  <link name="left_gripper_calib_link">
+  </link>
+  <velma_head parent="torso_link2">
+    <origin xyz="0 0.253 0.0" rpy="${-M_PI/2} 0 0"/>
+  </velma_head>
 </robot>

Commit message: head visualization

File: velma_description/defs/head.urdf.xacro (robot description, xacro)
@@ -99,4 +99,10 @@
         </material>
       </visual>
+      <visual>
+        <origin xyz="0 0 0.04219" rpy="0 0 0 " />
+        <geometry>
+          <mesh filename="package://velma_description/meshes/collision/head_top_collision.STL" />
+        </geometry>
+      </visual>
       <collision>
         <origin xyz="0 0 0.04219" rpy="0 0 0 " />
@@ -112,5 +118,11 @@
       </self_collision_checking>
       <self_collision_checking>
-        <origin xyz="0.05 0.18 0.0" rpy="0 0 0"/>
+        <origin xyz="-0.12 0.17 0.0" rpy="-1.57075 0 0"/>
+        <geometry>
+          <capsule radius="0.07" length="0.14"/>
+        </geometry>
+      </self_collision_checking>
+      <self_collision_checking>
+        <origin xyz="0.0 0.20 0.0" rpy="0 0 0"/>
         <geometry>
           <capsule radius="0.07" length="0.23"/>

Commit message: added missing inertia parameters

File: velma_description/defs/head.urdf.xacro (robot description, xacro)
@@ -27,4 +27,9 @@
         </geometry>
       </collision>
+      <inertial>
+        <mass value="0.2"/>
+        <origin rpy="0 0 0" xyz="0 0 0.0625"/>
+        <inertia ixx="0.000520833333333" ixy="0" ixz="0" iyy="0.000520833333333" iyz="0" izz="0.000520833333333"/>
+      </inertial>
     </link>
     <joint name="head_pan_motor_joint" type="fixed">
@@ -55,4 +60,9 @@
         </geometry>
       </self_collision_checking>
+      <inertial>
+        <mass value="0.2"/>
+        <origin rpy="0 0 0" xyz="0 0 0.0625"/>
+        <inertia ixx="0.000520833333333" ixy="0" ixz="0" iyy="0.000520833333333" iyz="0" izz="0.000520833333333"/>
+      </inertial>
     </link>
     <!-- pan -->
@@ -80,4 +90,9 @@
         </geometry>
       </collision>
+      <inertial>
+        <mass value="0.2"/>
+        <origin rpy="0 0 0" xyz="0 0 0.0625"/>
+        <inertia ixx="0.000520833333333" ixy="0" ixz="0" iyy="0.000520833333333" iyz="0" izz="0.000520833333333"/>
+      </inertial>
     </link>
     <!-- tilt -->
@@ -129,4 +144,9 @@
         </geometry>
       </self_collision_checking>
+      <inertial>
+        <mass value="0.2"/>
+        <origin rpy="0 0 0" xyz="0 0 0.0625"/>
+        <inertia ixx="0.000520833333333" ixy="0" ixz="0" iyy="0.000520833333333" iyz="0" izz="0.000520833333333"/>
+      </inertial>
     </link>
     <!-- sensors -->

File: velma_description/defs/torso.urdf.xacro (robot description, xacro)
@@ -31,4 +31,9 @@
       </self_collision_checking>
 -->
+      <inertial>
+        <mass value="2.0"/>
+        <origin rpy="0 0 0" xyz="0 -0.06 0.130"/>
+        <inertia ixx="0.0136666666667" ixy="0" ixz="0" iyy="0.003" iyz="0" izz="0.0118666666667"/>
+      </inertial>
     </link>
     <joint name="torso_0_joint" type="revolute">
@@ -77,4 +82,9 @@
         </geometry>
       </self_collision_checking>
+      <inertial>
+        <mass value="2.0"/>
+        <origin rpy="0 0 0" xyz="0 -0.06 0.130"/>
+        <inertia ixx="0.0136666666667" ixy="0" ixz="0" iyy="0.003" iyz="0" izz="0.0118666666667"/>
+      </inertial>
     </link>
   </macro>

File: velma_description/robots/velma.urdf.xacro (robot description, xacro)
@@ -21,5 +21,5 @@
   <link name="world" />
   <!-- static connection between the world frame and the map frame -->
-  <link name="map" />
+  <link name="map"/>
   <joint name="world_map_joint" type="fixed">
     <origin xyz="0 0 0" rpy="0 0 0"/>
@@ -63,4 +63,9 @@
       </geometry>
     </self_collision_checking>
+    <inertial>
+      <mass value="0.2"/>
+      <origin rpy="0 0 0" xyz="0 0 0.0625"/>
+      <inertia ixx="0.000520833333333" ixy="0" ixz="0" iyy="0.000520833333333" iyz="0" izz="0.000520833333333"/>
+    </inertial>
   </link>
   <joint name="left_gripper_mount_joint" type="fixed">
@@ -91,4 +96,9 @@
       </geometry>
     </self_collision_checking>
+    <inertial>
+      <mass value="0.2"/>
+      <origin rpy="0 0 0" xyz="0 0 0.0625"/>
+      <inertia ixx="0.000520833333333" ixy="0" ixz="0" iyy="0.000520833333333" iyz="0" izz="0.000520833333333"/>
+    </inertial>
   </link>
   <xacro:barret_hand prefix="right" parent="right_arm_7_link">
@@ -100,6 +110,5 @@
     <child link="right_gripper_calib_link"/>
   </joint>
-  <link name="right_gripper_calib_link">
-  </link>
+  <link name="right_gripper_calib_link"/>
   <joint name="right_gripper_calib_joint1" type="fixed">
     <origin xyz="${cal_right_gripper_calib_link1_x} ${cal_right_gripper_calib_link1_y} ${cal_right_gripper_calib_link1_z}" rpy="${cal_right_gripper_calib_link1_roll} ${cal_right_gripper_calib_link1_pitch} ${cal_right_gripper_calib_link1_yaw}"/>
@@ -107,6 +116,5 @@
     <child link="right_gripper_calib_link1"/>
   </joint>
-  <link name="right_gripper_calib_link1">
-  </link>
+  <link name="right_gripper_calib_link1"/>
   <joint name="right_gripper_calib_joint2" type="fixed">
     <origin xyz="${cal_right_gripper_calib_link2_x} ${cal_right_gripper_calib_link2_y} ${cal_right_gripper_calib_link2_z}" rpy="${cal_right_gripper_calib_link2_roll} ${cal_right_gripper_calib_link2_pitch} ${cal_right_gripper_calib_link2_yaw}"/>
@@ -114,6 +122,5 @@
     <child link="right_gripper_calib_link2"/>
   </joint>
-  <link name="right_gripper_calib_link2">
-  </link>
+  <link name="right_gripper_calib_link2"/>
   <xacro:barret_hand prefix="left" parent="left_arm_7_link">
     <origin xyz="-0.115 0.0 -0.078" rpy="0 ${-M_PI/2} 0"/>
@@ -124,6 +131,5 @@
     <child link="left_gripper_calib_link"/>
   </joint>
-  <link name="left_gripper_calib_link">
-  </link>
+  <link name="left_gripper_calib_link"/>
   <joint name="left_gripper_calib_joint1" type="fixed">
     <origin xyz="${cal_left_gripper_calib_link1_x} ${cal_left_gripper_calib_link1_y} ${cal_left_gripper_calib_link1_z}" rpy="${cal_left_gripper_calib_link1_roll} ${cal_left_gripper_calib_link1_pitch} ${cal_left_gripper_calib_link1_yaw}"/>
@@ -131,6 +137,5 @@
     <child link="left_gripper_calib_link1"/>
   </joint>
-  <link name="left_gripper_calib_link1">
-  </link>
+  <link name="left_gripper_calib_link1"/>
   <joint name="left_gripper_calib_joint2" type="fixed">
     <origin xyz="${cal_left_gripper_calib_link2_x} ${cal_left_gripper_calib_link2_y} ${cal_left_gripper_calib_link2_z}" rpy="${cal_left_gripper_calib_link2_roll} ${cal_left_gripper_calib_link2_pitch} ${cal_left_gripper_calib_link2_yaw}"/>
@@ -138,6 +143,5 @@
     <child link="left_gripper_calib_link2"/>
   </joint>
-  <link name="left_gripper_calib_link2">
-  </link>
+  <link name="left_gripper_calib_link2"/>
   <head_camera parent="left_arm_7_link" name="left_hand_camera">
       <origin xyz="${cal_left_hand_camera_joint_x} ${cal_left_hand_camera_joint_y} ${cal_left_hand_camera_joint_z}"

Commit message: impoved damping and inertia parameters in urdf

File: velma_description/defs/head.urdf.xacro (robot description, xacro)
@@ -73,4 +73,5 @@
       <child link="head_pan_link"/>
       <limit lower="-1.57" upper="1.57" effort="100" velocity="1.57"/>
+      <dynamics damping="0.1"/>
     </joint>
     <link name="head_pan_link">
@@ -103,4 +104,5 @@
       <child link="head_tilt_link"/>
       <limit lower="-1.57" upper="1.57" effort="100" velocity="100"/>
+      <dynamics damping="0.1"/>
     </joint>
     <link name="head_tilt_link">

File: velma_description/defs/torso.urdf.xacro (robot description, xacro)
@@ -32,7 +32,7 @@
 -->
       <inertial>
-        <mass value="2.0"/>
+        <mass value="30.0"/>
         <origin rpy="0 0 0" xyz="0 -0.06 0.130"/>
-        <inertia ixx="0.0136666666667" ixy="0" ixz="0" iyy="0.003" iyz="0" izz="0.0118666666667"/>
+        <inertia ixx="0.9" ixy="0" ixz="0" iyy="0.9" iyz="0" izz="1.35"/>
       </inertial>
     </link>
@@ -43,4 +43,5 @@
       <parent link="torso_base"/>
       <child link="torso_link0"/>
+      <dynamics damping="10.0"/>
     </joint>
     <link name="torso_link0">
@@ -83,7 +84,7 @@
       </self_collision_checking>
       <inertial>
-        <mass value="2.0"/>
+        <mass value="30.0"/>
         <origin rpy="0 0 0" xyz="0 -0.06 0.130"/>
-        <inertia ixx="0.0136666666667" ixy="0" ixz="0" iyy="0.003" iyz="0" izz="0.0118666666667"/>
+        <inertia ixx="3.175" ixy="0" ixz="0" iyy="3.175" iyz="0" izz="1.35"/>
       </inertial>
     </link>

Commit message: added self_collide tag for velma links (for gazebo)

File: velma_description/defs/head.urdf.xacro (robot description, xacro)
@@ -97,4 +97,8 @@
       </inertial>
     </link>
+    <gazebo reference="head_pan_link">
+      <turnGravityOff>false</turnGravityOff>
+      <selfCollide>true</selfCollide>
+    </gazebo>
     <!-- tilt -->
     <joint name="head_tilt_joint" type="revolute">
@@ -152,4 +156,8 @@
       </inertial>
     </link>
+    <gazebo reference="head_tilt_link">
+      <turnGravityOff>false</turnGravityOff>
+      <selfCollide>true</selfCollide>
+    </gazebo>
     <!-- sensors -->
     <head_camera parent="head_tilt_link" name="stereo_left">

File: velma_description/defs/torso.urdf.xacro (robot description, xacro)
@@ -20,4 +20,5 @@
         </material>
       </visual>
+<!--
       <collision>
         <origin xyz="0 0 0.1" rpy="0 0 0"/>
@@ -26,4 +27,5 @@
         </geometry>
       </collision>
+-->
 <!--
       <self_collision_checking>
@@ -40,4 +42,8 @@
       </inertial>
     </link>
+    <gazebo reference="torso_base">
+      <turnGravityOff>false</turnGravityOff>
+      <selfCollide>true</selfCollide>
+    </gazebo>
     <joint name="torso_0_joint" type="revolute">
       <origin xyz="0 0 0.1" rpy="0 0 0"/>
@@ -92,4 +98,8 @@
       </inertial>
     </link>
+    <gazebo reference="torso_link0">
+      <turnGravityOff>false</turnGravityOff>
+      <selfCollide>true</selfCollide>
+    </gazebo>
   </xacro:macro>
 </robot>

File: velma_description/robots/velma.urdf.xacro (robot description, xacro)
@@ -166,4 +166,5 @@
   <gazebo reference="right_gripper_mount_link">
     <turnGravityOff>false</turnGravityOff>
+    <selfCollide>true</selfCollide>
   </gazebo>
   <joint name="left_gripper_mount_joint" type="fixed">
@@ -202,8 +203,13 @@
   <gazebo reference="left_gripper_mount_link">
     <turnGravityOff>false</turnGravityOff>
+    <selfCollide>true</selfCollide>
   </gazebo>
   <xacro:barret_hand prefix="right" parent="right_arm_7_link" with_optoforce="false">
     <origin xyz="0.115 0.0 -0.078" rpy="0 ${M_PI/2} 0"/>
   </xacro:barret_hand>
+  <xacro:barret_hand prefix="left" parent="left_arm_7_link" with_optoforce="true">
+    <origin xyz="-0.115 0.0 -0.078" rpy="0 ${-M_PI/2} 0"/>
+  </xacro:barret_hand>
+<!--
   <joint name="right_gripper_calib_joint" type="fixed">
     <origin xyz="${cal_right_gripper_calib_link_x} ${cal_right_gripper_calib_link_y} ${cal_right_gripper_calib_link_z}" rpy="0 0 0"/>
@@ -224,7 +230,6 @@
   </joint>
   <link name="right_gripper_calib_link2"/>
-  <xacro:barret_hand prefix="left" parent="left_arm_7_link" with_optoforce="true">
-    <origin xyz="-0.115 0.0 -0.078" rpy="0 ${-M_PI/2} 0"/>
-  </xacro:barret_hand>
+-->
+<!--
   <joint name="left_gripper_calib_joint" type="fixed">
     <origin xyz="${cal_left_gripper_calib_link_x} ${cal_left_gripper_calib_link_y} ${cal_left_gripper_calib_link_z}" rpy="0 0 0"/>
@@ -249,4 +254,5 @@
               rpy="${cal_left_hand_camera_joint_roll} ${cal_left_hand_camera_joint_pitch} ${cal_left_hand_camera_joint_yaw}"/>
   </head_camera>
+  -->
   <velma_head parent="torso_link0">
     <origin xyz="${cal_head_base_joint_x} ${cal_head_base_joint_y} ${cal_head_base_joint_z}" rpy="${cal_head_base_joint_roll} ${cal_head_base_joint_pitch} ${cal_head_base_joint_yaw}"/>

Commit message: simpler visual geometries

File: velma_description/defs/head.urdf.xacro (robot description, xacro)
@@ -15,5 +15,5 @@
         <origin xyz="0 0 0.0" rpy="0 0 0" />
         <geometry>
-          <mesh filename="package://velma_description/meshes/head_base.STL" />
+          <mesh filename="package://velma_description/meshes/head_base_simplified.STL" />
         </geometry>
         <material name="torso_gray">
@@ -42,5 +42,5 @@
         <origin xyz="0 0 0" rpy="0 0 0" />
         <geometry>
-          <mesh filename="package://velma_description/meshes/head_pan.STL" />
+          <mesh filename="package://velma_description/meshes/head_pan_simplified.STL" />
         </geometry>
         <material name="torso_gray">
@@ -79,5 +79,5 @@
         <origin xyz="0 0 0" rpy="0 0 0" />
         <geometry>
-          <mesh filename="package://velma_description/meshes/head_tilt.STL" />
+          <mesh filename="package://velma_description/meshes/head_tilt_simplified.STL" />
         </geometry>
         <material name="torso_gray">
@@ -114,5 +114,5 @@
         <origin xyz="0 0 0.04219" rpy="0 0 0" />
         <geometry>
-          <mesh filename="package://velma_description/meshes/head_top.STL" />
+          <mesh filename="package://velma_description/meshes/head_top_simplified.STL" />
         </geometry>
         <material name="torso_gray">

File: velma_description/defs/torso.urdf.xacro (robot description, xacro)
@@ -55,4 +55,5 @@
     </joint>
     <link name="torso_link0">
+<!--
       <visual>
         <origin xyz="0 0 0.219" rpy="0.0 0 0" />
@@ -80,4 +81,14 @@
         <material name="torso_asm">
           <color rgba="1.0 0.487 0 1.0"/>
+        </material>
+      </visual>
+-->
+      <visual>
+        <origin xyz="0 0 0.52" rpy="0 0 0"/>
+        <geometry>
+          <mesh filename="package://velma_description/meshes/collision/torso0_collision.stl" />
+        </geometry>
+        <material name="torso_base">
+          <color rgba="0.7 0.7 0.7 1"/>
         </material>
       </visual>

File: velma_description/robots/velma.urdf.xacro (robot description, xacro)
@@ -182,5 +182,5 @@
       <sensor type="depth" name="openni_camera_camera">
         <always_on>0</always_on>
-        <update_rate>30.0</update_rate>
+        <update_rate>15.0</update_rate>
         <visualize>false</visualize>
         <camera>
@@ -250,5 +250,5 @@
       <origin xyz="0 0 0" rpy="0.0 0 0" />
       <geometry>
-        <mesh filename="package://velma_description/meshes/gripper_mount.STL" />
+        <mesh filename="package://velma_description/meshes/gripper_mount_simplified.STL" />
       </geometry>
       <material name="Orange"/>
@@ -311,5 +311,5 @@
       <origin xyz="0 0 0" rpy="0.0 0 0" />
       <geometry>
-        <mesh filename="package://velma_description/meshes/gripper_mount.STL" />
+        <mesh filename="package://velma_description/meshes/gripper_mount_simplified.STL" />
       </geometry>
       <material name="Orange"/>
