Commit message: patch for bug in KDL/URDF

File: velma_description/defs/head.urdf.xacro (robot description, xacro)
@@ -103,11 +103,21 @@
     <!-- tilt -->
     <joint name="head_tilt_joint" type="revolute">
-      <origin xyz="0 0 0.048" rpy="1.57 0.0 0" />
-      <axis xyz="0 0 -1"/>
+      <origin xyz="0 0 0.048" rpy="0 0 0" />
+      <axis xyz="0 1 0"/>
       <parent link="head_pan_link"/>
+      <child link="head_tilt_link_dummy"/>
+      <limit lower="-1.57" upper="1.57" effort="100" velocity="100"/>
+      <dynamics damping="0.1"/>
+    </joint>
+    <!-- PATCH: The added dummy joint and link is a bugfix for KDL issue with rotated joints -->
+    <link name="head_tilt_link_dummy"/>
+    <joint name="head_tilt_joint_dummy" type="fixed">
+      <origin xyz="0 0 0.0" rpy="${M_PI/2} 0 0" />
+      <parent link="head_tilt_link_dummy"/>
       <child link="head_tilt_link"/>
       <limit lower="-1.57" upper="1.57" effort="100" velocity="100"/>
       <dynamics damping="0.1"/>
     </joint>
+    <!-- end of PATCH -->
     <link name="head_tilt_link">
       <visual>

Commit message: added dart collision model using spheres and boxes only

File: velma_description/defs/head.urdf.xacro (robot description, xacro)
@@ -4,4 +4,6 @@
                         xmlns:sensor="http://playerstage.sourceforge.net/gazebo/xmlschema/#sensor"
                         xmlns:xacro="http://www.ros.org/wiki/xacro">
+  <xacro:arg name="collision_detector" default="fcl"/>
+  <xacro:property name="collision_detector" value="$(arg collision_detector)"/>
   <xacro:include filename="$(find velma_description)/defs/camera.urdf.xacro" />
   <xacro:macro name="velma_head" params="parent *origin">
@@ -21,10 +23,20 @@
         </material>
       </visual>
-      <collision>
-        <origin xyz="0 0 0.0" rpy="0 0 0" />
-        <geometry>
-          <mesh filename="package://velma_description/meshes/collision/head_base_collision.STL" />
-        </geometry>
-      </collision>
+      <xacro:if value="${collision_detector == 'fcl'}">
+        <collision>
+          <origin xyz="0 0 0.0" rpy="0 0 0" />
+          <geometry>
+            <mesh filename="package://velma_description/meshes/collision/head_base_collision.STL" />
+          </geometry>
+        </collision>
+      </xacro:if>
+      <xacro:if value="${collision_detector == 'dart'}">
+        <collision>
+          <origin xyz="0 0 0" rpy="0 0 0"/>
+          <geometry>
+            <box size="0.244826734066 0.069836191833 0.0559380054474"/>
+          </geometry>
+        </collision>
+      </xacro:if>
       <inertial>
         <mass value="0.2"/>
@@ -136,10 +148,26 @@
         </geometry>
       </visual>
-      <collision>
-        <origin xyz="0 0 0.04219" rpy="0 0 0 " />
-        <geometry>
-          <mesh filename="package://velma_description/meshes/collision/head_top_collision.STL" />
-        </geometry>
-      </collision>
+      <xacro:if value="${collision_detector == 'fcl'}">
+        <collision>
+          <origin xyz="0 0 0.04219" rpy="0 0 0 " />
+          <geometry>
+            <mesh filename="package://velma_description/meshes/collision/head_top_collision.STL" />
+          </geometry>
+        </collision>
+      </xacro:if>
+      <xacro:if value="${collision_detector == 'dart'}">
+        <collision>
+          <origin xyz="-0.0568619705737 0.1684935987 0" rpy="0 0 0"/>
+          <geometry>
+            <box size="0.197051048279 0.218739390373 0.121755480766"/>
+          </geometry>
+        </collision>
+        <collision>
+          <origin xyz="0.00178006081842 0.200341254473 0" rpy="0 0 0"/>
+          <geometry>
+            <box size="0.0787106156349 0.0698484331369 0.306180119514"/>
+          </geometry>
+        </collision>
+      </xacro:if>
       <self_collision_checking>
         <origin xyz="0.0 0.12 0.0" rpy="-1.57075 0 0"/>

File: velma_description/defs/torso.urdf.xacro (robot description, xacro)
@@ -4,4 +4,6 @@
                         xmlns:sensor="http://playerstage.sourceforge.net/gazebo/xmlschema/#sensor"
                         xmlns:xacro="http://www.ros.org/wiki/xacro">
+  <xacro:arg name="collision_detector" default="fcl"/>
+  <xacro:property name="collision_detector" value="$(arg collision_detector)"/>
   <xacro:macro name="velma_torso" params="*origin">
     <link name="world" />
@@ -132,10 +134,32 @@
         </material>
       </visual>
-      <collision>
-        <origin xyz="0 0 0.52" rpy="0 0 0"/>
-        <geometry>
-          <mesh filename="package://velma_description/meshes/collision/torso0_collision.stl" />
-        </geometry>
-      </collision>
+      <xacro:if value="${collision_detector == 'fcl'}">
+        <collision>
+          <origin xyz="0 0 0.52" rpy="0 0 0"/>
+          <geometry>
+            <mesh filename="package://velma_description/meshes/collision/torso0_collision.stl" />
+          </geometry>
+        </collision>
+      </xacro:if>
+      <xacro:if value="${collision_detector == 'dart'}">
+        <collision>
+          <origin xyz="0 0 0.968570022583" rpy="0 0 0"/>
+          <geometry>
+            <box size="0.30822044611 0.276354163885 0.45334654808"/>
+          </geometry>
+        </collision>
+        <collision>
+          <origin xyz="0 0 1.18425571918" rpy="${M_PI/4} 0 0"/>
+          <geometry>
+            <box size="0.316696882248 0.19 0.19"/>
+          </geometry>
+        </collision>
+        <collision>
+          <origin xyz="-0.0265109799802 0 0.505967736244" rpy="0 0 0"/>
+          <geometry>
+            <box size="0.353161275387 0.255815982819 0.5"/>
+          </geometry>
+        </collision>
+      </xacro:if>
       <self_collision_checking>
         <origin xyz="0 0.0 0.8" rpy="0 0 0"/>

File: velma_description/robots/velma.urdf.xacro (robot description, xacro)
@@ -5,8 +5,10 @@
                         xmlns:xacro="http://www.ros.org/wiki/xacro"
 	 name="velma">
-  <xacro:arg name="collision_model_full" default="true"/>
-  <xacro:arg name="collision_model_simplified" default="false"/>
+  <xacro:arg name="collision_model_full" default="false"/>
+  <xacro:arg name="collision_model_simplified" default="true"/>
   <xacro:arg name="collision_model_enlargement" default="0.0"/>
   <xacro:arg name="collision_model_no_hands" default="false"/>
+  <xacro:arg name="collision_detector" default="fcl"/>
+  <xacro:property name="collision_detector" value="$(arg collision_detector)"/>
   <xacro:arg name="subsystem_xml" default="false"/>
   <xacro:arg name="xml_file_re_body" default=""/>
@@ -72,4 +74,5 @@
     <plugin name="rtt_gazebo" filename="librtt_gazebo_deployer.so">
       <isolated/>
+      <collision_detector>${collision_detector}</collision_detector>
       <xacro:if value="$(arg subsystem_xml)">
         <subsystem_xml>
@@ -362,10 +365,32 @@
     </visual>
     <xacro:unless value="$(arg collision_model_no_hands)">
-      <collision>
-        <origin xyz="0 0 0" rpy="0 0 0"/>
-        <geometry>
-          <mesh filename="package://velma_description/meshes/collision/gripper_mount_collision2.STL"/>
-        </geometry>
-      </collision>
+      <xacro:if value="${collision_detector == 'fcl'}">
+        <collision>
+          <origin xyz="0 0 0" rpy="0 0 0"/>
+          <geometry>
+            <mesh filename="package://velma_description/meshes/collision/gripper_mount_collision2.STL"/>
+          </geometry>
+        </collision>
+      </xacro:if>
+      <xacro:if value="${collision_detector == 'dart'}">
+        <collision>
+          <origin xyz="0.00848898105323 0.0 0.0221745967865" rpy="0 0 0"/>
+          <geometry>
+            <box size="0.110316336155 0.0795853585005 0.0497657060623"/>
+          </geometry>
+        </collision>
+        <collision>
+          <origin xyz="0.0838752761483 0 -0.0117062330246" rpy="0 0.822849241182 0"/>
+          <geometry>
+            <box size="0.068020761013 0.0795853585005 0.025487780571"/>
+          </geometry>
+        </collision>
+        <collision>
+          <origin xyz="0.102500602603 0 -0.0791217014194" rpy="0 0 0"/>
+          <geometry>
+            <box size="0.0187338590622 0.0816289409995 0.100000023842"/>
+          </geometry>
+        </collision>
+      </xacro:if>
     </xacro:unless>
     <self_collision_checking>
@@ -417,10 +442,32 @@
     </visual>
     <xacro:unless value="$(arg collision_model_no_hands)">
-      <collision>
-        <origin xyz="0 0 0" rpy="0 0 0"/>
-        <geometry>
-          <mesh filename="package://velma_description/meshes/collision/gripper_mount_collision2.STL"/>
-        </geometry>
-      </collision>
+      <xacro:if value="${collision_detector == 'fcl'}">
+        <collision>
+          <origin xyz="0 0 0" rpy="0 0 0"/>
+          <geometry>
+            <mesh filename="package://velma_description/meshes/collision/gripper_mount_collision2.STL"/>
+          </geometry>
+        </collision>
+      </xacro:if>
+      <xacro:if value="${collision_detector == 'dart'}">
+        <collision>
+          <origin xyz="0.00848898105323 0.0 0.0221745967865" rpy="0 0 0"/>
+          <geometry>
+            <box size="0.110316336155 0.0795853585005 0.0497657060623"/>
+          </geometry>
+        </collision>
+        <collision>
+          <origin xyz="0.0838752761483 0 -0.0117062330246" rpy="0 0.822849241182 0"/>
+          <geometry>
+            <box size="0.068020761013 0.0795853585005 0.025487780571"/>
+          </geometry>
+        </collision>
+        <collision>
+          <origin xyz="0.102500602603 0 -0.0791217014194" rpy="0 0 0"/>
+          <geometry>
+            <box size="0.0187338590622 0.0816289409995 0.100000023842"/>
+          </geometry>
+        </collision>
+      </xacro:if>
     </xacro:unless>
     <self_collision_checking>

Commit message: updated limits for head

File: velma_description/defs/head.urdf.xacro (robot description, xacro)
@@ -119,5 +119,5 @@
       <parent link="head_pan_link"/>
       <child link="head_tilt_link_dummy"/>
-      <limit lower="-1.57" upper="1.57" effort="100" velocity="100"/>
+      <limit lower="-1.0" upper="1.3" effort="100" velocity="100"/>
       <dynamics damping="0.1"/>
     </joint>

Commit message: removed detailed collision geometries for head

File: velma_description/defs/head.urdf.xacro (robot description, xacro)
@@ -60,4 +60,5 @@
         </material>
       </visual>
+<!--
       <collision>
         <origin xyz="0 0 0.0308" rpy="0 0 0" />
@@ -72,4 +73,5 @@
         </geometry>
       </self_collision_checking>
+-->
       <inertial>
         <mass value="0.2"/>
@@ -97,5 +99,6 @@
         </material>
       </visual>
-      <collision>
+<!--
+       <collision>
         <origin xyz="0 -0.00921 0.04463" rpy="0 0 0" />
         <geometry>
@@ -103,4 +106,5 @@
         </geometry>
       </collision>
+ -->
       <inertial>
         <mass value="0.2"/>
@@ -148,4 +152,5 @@
         </geometry>
       </visual>
+<!--
       <xacro:if value="${collision_detector == 'fcl'}">
         <collision>
@@ -188,4 +193,5 @@
         </geometry>
       </self_collision_checking>
+ -->
       <inertial>
         <mass value="0.2"/>
