Commit message: added collision description

File: velma_description/defs/torso.urdf.xacro (robot description, xacro)
@@ -44,4 +44,27 @@
         </material>
       </visual>
+      <self_collision_checking>
+        <origin xyz="0 0.0 0.4" rpy="0 0 0"/>
+        <geometry>
+          <capsule radius="0.20" length="0.8"/>
+        </geometry>
+      </self_collision_checking>
+      <self_collision_checking>
+        <origin xyz="0 0 0" rpy="0 0 0"/>
+        <geometry>
+          <convex>
+            <point xyz="0.15 0.14 0.8" frame="torso_link0"/>
+            <point xyz="-0.15 0.14 0.8" frame="torso_link0"/>
+            <point xyz="-0.15 -0.14 0.8" frame="torso_link0"/>
+            <point xyz="0.15 -0.14 0.8" frame="torso_link0"/>
+            <point xyz="0.15 0.08 0.14" frame="torso_link2"/>
+            <point xyz="-0.15 0.08 0.14" frame="torso_link2"/>
+            <point xyz="-0.15 0.08 -0.14" frame="torso_link2"/>
+            <point xyz="0.15 0.08 -0.14" frame="torso_link2"/>
+            <point xyz="0.15 0.3 0" frame="torso_link2"/>
+            <point xyz="-0.15 0.3 0" frame="torso_link2"/>
+          </convex>
+        </geometry>
+      </self_collision_checking>
     </link>
     <joint name="torso_1_joint" type="revolute">

Commit message: complete collision model for Velma

File: velma_description/defs/torso.urdf.xacro (robot description, xacro)
@@ -17,4 +17,10 @@
         </material>
       </visual>
+      <collision>
+        <origin xyz="0 0 0" rpy="0 0 0"/>
+        <geometry>
+          <mesh filename="package://velma_description/meshes/collision/torso_base_collision.STL" />
+        </geometry>
+      </collision>
       <self_collision_checking>
         <origin xyz="-0.2 0.0 0.6" rpy="1.57075 0 0"/>

Commit message: self-collision model

File: velma_description/defs/torso.urdf.xacro (robot description, xacro)
@@ -54,9 +54,10 @@
       </collision>
       <self_collision_checking>
-        <origin xyz="0 0.0 0.4" rpy="0 0 0"/>
+        <origin xyz="0 0.0 0.8" rpy="0 0 0"/>
         <geometry>
-          <capsule radius="0.20" length="0.8"/>
+          <capsule radius="0.20" length="1.0"/>
         </geometry>
       </self_collision_checking>
+<!--
       <self_collision_checking>
         <origin xyz="0 0 0" rpy="0 0 0"/>
@@ -76,4 +77,5 @@
         </geometry>
       </self_collision_checking>
+-->
     </link>
     <joint name="torso_1_joint" type="revolute">

Commit message: new velma kinematics structure.

File: velma_description/defs/torso.urdf.xacro (robot description, xacro)
@@ -47,4 +47,11 @@
         </material>
       </visual>
+      <visual>
+        <origin xyz="0 0.0 1.055" rpy="0 0 0.0" />
+        <geometry>
+          <mesh filename="package://velma_description/meshes/top_base_asm.STL" />
+        </geometry>
+        <material name="Orange"/>
+      </visual>
       <collision>
         <origin xyz="-0.03338 0 0.519" rpy="0 0 0"/>
@@ -59,106 +66,4 @@
         </geometry>
       </self_collision_checking>
-<!--
-      <self_collision_checking>
-        <origin xyz="0 0 0" rpy="0 0 0"/>
-        <geometry>
-          <convex>
-            <point xyz="0.15 0.14 0.8" frame="torso_link0"/>
-            <point xyz="-0.15 0.14 0.8" frame="torso_link0"/>
-            <point xyz="-0.15 -0.14 0.8" frame="torso_link0"/>
-            <point xyz="0.15 -0.14 0.8" frame="torso_link0"/>
-            <point xyz="0.15 0.08 0.14" frame="torso_link2"/>
-            <point xyz="-0.15 0.08 0.14" frame="torso_link2"/>
-            <point xyz="-0.15 0.08 -0.14" frame="torso_link2"/>
-            <point xyz="0.15 0.08 -0.14" frame="torso_link2"/>
-            <point xyz="0.15 0.3 0" frame="torso_link2"/>
-            <point xyz="-0.15 0.3 0" frame="torso_link2"/>
-          </convex>
-        </geometry>
-      </self_collision_checking>
--->
-    </link>
-    <joint name="torso_1_joint" type="revolute">
-      <origin xyz="0 0 0.80" rpy="${M_PI/2} 0 0"/>
-      <axis xyz="0 0 -1"/>
-      <limit lower="${-105 * M_PI/180}" upper="${-M_PI/4}" effort="100" velocity="100"/>
-      <parent link="torso_link0"/>
-      <child link="torso_link1"/>
-    </joint>
-    <link name="torso_link1">
-    </link>
-    <joint name="torso_1_joint_viz1" type="revolute">
-      <origin xyz="0.09 0 0.80" rpy="${M_PI/2} 0 0"/>
-      <axis xyz="0 0 -1"/>
-      <limit lower="${-105 * M_PI/180}" upper="${-M_PI/4}" effort="100" velocity="100"/>
-      <mimic joint="torso_1_joint" multiplier="1"/>
-      <parent link="torso_link0"/>
-      <child link="torso_link1_viz1"/>
-    </joint>
-    <link name="torso_link1_viz1">
-      <visual>
-        <origin xyz="0 0 -0.09875" rpy="${-M_PI/2} 0 ${-M_PI/2}" />
-        <geometry>
-          <mesh filename="package://velma_description/meshes/connector.STL" />
-        </geometry>
-        <material name="torso_gray">
-          <color rgba="0.5 0.5 0.5 1"/>
-        </material>
-      </visual>
-      <collision>
-        <origin xyz="0 0 -0.09875" rpy="${-M_PI/2} 0 ${-M_PI/2}" />
-        <geometry>
-          <mesh filename="package://velma_description/meshes/collision/connector2_collision.STL" />
-        </geometry>
-      </collision>
-    </link>
-    <joint name="torso_1_joint_viz2" type="revolute">
-      <origin xyz="-0.13 0 0.80" rpy="${M_PI/2} 0 0"/>
-      <axis xyz="0 0 -1"/>
-      <limit lower="${-105 * M_PI/180}" upper="${-M_PI/4}" effort="100" velocity="100"/>
-      <mimic joint="torso_1_joint" multiplier="1"/>
-      <parent link="torso_link0"/>
-      <child link="torso_link1_viz2"/>
-    </joint>
-    <link name="torso_link1_viz2">
-      <visual>
-        <origin xyz="0 0 -0.09875" rpy="${-M_PI/2} 0 ${-M_PI/2}" />
-        <geometry>
-          <mesh filename="package://velma_description/meshes/connector.STL" />
-        </geometry>
-        <material name="torso_gray">
-          <color rgba="0.5 0.5 0.5 1"/>
-        </material>
-      </visual>
-      <collision>
-        <origin xyz="0 0 -0.09875" rpy="${-M_PI/2} 0 ${-M_PI/2}" />
-        <geometry>
-          <mesh filename="package://velma_description/meshes/collision/connector_collision.STL" />
-        </geometry>
-      </collision>
-    </link>
-    <joint name="torso_2_joint" type="revolute">
-      <origin xyz="0.375 0 0" rpy="0 0 0"/>
-      <axis xyz="0 0 -1"/>
-      <limit lower="-1.57" upper="1.57" effort="100" velocity="100"/>
-      <mimic joint="torso_1_joint" multiplier="-1"/>
-      <parent link="torso_link1"/>
-      <child link="torso_link2"/>
-    </joint>
-    <link name="torso_link2">
-      <visual>
-        <origin xyz="0 0.0 0" rpy="${-M_PI/2.0} 0 0.0" />
-        <geometry>
-          <mesh filename="package://velma_description/meshes/top_base_asm.STL" />
-        </geometry>
-        <material name="Orange"/>
-      </visual>
-      <collision>
-        <origin xyz="0 0.0 0" rpy="${-M_PI/2.0} 0 0.0" />
-        <geometry>
-          <mesh filename="package://velma_description/meshes/collision/top_base_asm_collision.STL" />
-        </geometry>
-        <material name="Orange"/>
-      </collision>
     </link>
   </macro>

File: velma_description/robots/velma.urdf.xacro (robot description, xacro)
@@ -30,8 +30,8 @@
     <origin xyz="0 0 0.1" rpy="0 0 0"/>
   </velma_torso>
-  <kuka_lwr_arm parent="torso_link2" name="right" right="1">
-    <origin xyz="0 0.1641 0.07943" rpy="${-M_PI/6} 0 0"/>
+  <kuka_lwr_arm parent="torso_link0" name="right" right="1">
+    <origin xyz="0 -0.000188676 1.17335" rpy="0 ${-M_PI/3} ${M_PI/2}"/>
   </kuka_lwr_arm>
-  <kuka_lwr_arm parent="torso_link2" name="left" right="1">
+  <kuka_lwr_arm parent="torso_link0" name="left" right="1">
     <origin xyz="${cal_torso_link2_left_arm_base_joint_x} ${cal_torso_link2_left_arm_base_joint_y} ${cal_torso_link2_left_arm_base_joint_z}" rpy="${cal_torso_link2_left_arm_base_joint_roll} ${cal_torso_link2_left_arm_base_joint_pitch} ${cal_torso_link2_left_arm_base_joint_yaw}"/>
   </kuka_lwr_arm>
@@ -144,5 +144,5 @@
               rpy="${cal_left_hand_camera_joint_roll} ${cal_left_hand_camera_joint_pitch} ${cal_left_hand_camera_joint_yaw}"/>
   </head_camera>
-  <velma_head parent="torso_link2">
+  <velma_head parent="torso_link0">
     <origin xyz="${cal_head_base_joint_x} ${cal_head_base_joint_y} ${cal_head_base_joint_z}" rpy="${cal_head_base_joint_roll} ${cal_head_base_joint_pitch} ${cal_head_base_joint_yaw}"/>
   </velma_head>

Commit message: base = world

File: velma_description/defs/torso.urdf.xacro (robot description, xacro)
@@ -33,5 +33,5 @@
     </link>
     <joint name="torso_0_joint" type="revolute">
-      <origin xyz="0 0 0.0" rpy="0 0 0"/>
+      <origin xyz="0 0 0.1" rpy="0 0 0"/>
       <axis xyz="0 0 1"/>
       <limit lower="-1.57" upper="1.57" effort="100" velocity="100"/>

File: velma_description/robots/velma.urdf.xacro (robot description, xacro)
@@ -28,5 +28,5 @@
   </joint>
   <velma_torso parent="world" >
-    <origin xyz="0 0 0.1" rpy="0 0 0"/>
+    <origin xyz="0 0 0" rpy="0 0 0"/>
   </velma_torso>
   <kuka_lwr_arm parent="torso_link0" name="right" right="1">

Commit message: torso visualization for new kinematics

File: velma_description/defs/torso.urdf.xacro (robot description, xacro)
@@ -9,5 +9,5 @@
     <link name="torso_base">
       <visual>
-        <origin xyz="0 0 0" rpy="0.0 0 0" />
+        <origin xyz="0 0 0.1" rpy="0.0 0 0" />
         <geometry>
           <mesh filename="package://velma_description/meshes/torso_base.STL" />
@@ -18,5 +18,5 @@
       </visual>
       <collision>
-        <origin xyz="0 0 0" rpy="0 0 0"/>
+        <origin xyz="0 0 0.1" rpy="0 0 0"/>
         <geometry>
           <mesh filename="package://velma_description/meshes/collision/torso_base_collision.STL" />
@@ -50,4 +50,13 @@
       </visual>
       <visual>
+        <origin xyz="-0.01 0 0.93" rpy="0.0 0 0" />
+        <geometry>
+          <box size="0.28 0.24 0.32" />
+        </geometry>
+        <material name="torso_base">
+          <color rgba="0.5 0.5 0.5 1"/>
+        </material>
+      </visual>
+      <visual>
         <origin xyz="0 0.0 1.055" rpy="0 0 0.0" />
         <geometry>

Commit message: added collision mesh for torso

File: velma_description/defs/torso.urdf.xacro (robot description, xacro)
@@ -72,7 +72,7 @@
       </visual>
       <collision>
-        <origin xyz="-0.03338 0 0.519" rpy="0 0 0"/>
+        <origin xyz="0 0 0.52" rpy="0 0 0"/>
         <geometry>
-          <box size="0.34 0.3 0.6"/>
+          <mesh filename="package://velma_description/meshes/collision/torso0_collision.stl" />
         </geometry>
       </collision>

Commit message: added imu case in urdf

File: velma_description/defs/torso.urdf.xacro (robot description, xacro)
@@ -78,5 +78,7 @@
           <mesh filename="package://velma_description/meshes/top_base_asm.STL" />
         </geometry>
-        <material name="Orange"/>
+        <material name="torso_asm">
+          <color rgba="1.0 0.487 0 1.0"/>
+        </material>
       </visual>
       <collision>

File: velma_description/robots/velma.urdf.xacro (robot description, xacro)
@@ -20,9 +20,9 @@
   <xacro:arg name="xml_file_re_head" default=""/>
   <xacro:arg name="use_gazebo_kinect" default="false"/>
+  <xacro:include filename="$(find lwr_defs)/defs/materials.xml"/>
   <xacro:include filename="$(find velma_description)/calibration/default_cal.xml"/>
   <xacro:include filename="$(find velma_description)/defs/torso.urdf.xacro"/>
   <xacro:include filename="$(find velma_description)/defs/head.urdf.xacro" />
   <xacro:include filename="$(find lwr_defs)/defs/kuka_lwr_arm_defs.xml"/>
-  <xacro:include filename="$(find lwr_defs)/defs/materials.xml"/>
   <xacro:include filename="$(find barrett_hand_defs)/defs/barret_hand.urdf.xacro"/>
 <!--
@@ -186,6 +186,6 @@
           <horizontal_fov>1.047</horizontal_fov>
           <image>
-            <width>640</width>
-            <height>480</height>
+            <width>800</width>
+            <height>600</height>
             <format>B8G8R8</format>
           </image>
@@ -255,4 +255,11 @@
       <material name="Orange"/>
     </visual>
+    <visual>
+      <origin xyz="0 0 0" rpy="0.0 0 0" />
+      <geometry>
+        <mesh filename="package://velma_description/meshes/imu_case_right.stl" />
+      </geometry>
+      <material name="Orange"/>
+    </visual>
     <xacro:unless value="$(arg collision_model_no_hands)">
       <collision>

Commit message: added collision capsule for torso back element

File: velma_description/defs/torso.urdf.xacro (robot description, xacro)
@@ -94,4 +94,10 @@
         </geometry>
       </self_collision_checking>
+      <self_collision_checking>
+        <origin xyz="-0.1 0.0 0.45" rpy="0 0 0"/>
+        <geometry>
+          <capsule radius="0.18" length="0.4"/>
+        </geometry>
+      </self_collision_checking>
       <inertial>
         <mass value="30.0"/>
