Commit message: added mobile base

File: velma_description/defs/torso.urdf.xacro (robot description, xacro)
@@ -4,8 +4,9 @@
                         xmlns:sensor="http://playerstage.sourceforge.net/gazebo/xmlschema/#sensor"
                         xmlns:xacro="http://www.ros.org/wiki/xacro">
-  <xacro:macro name="velma_torso" params="parent *origin">
+  <xacro:macro name="velma_torso" params="*origin">
+    <link name="world" />
     <joint name="torso_base_joint" type="fixed">
       <xacro:insert_block name="origin" />
-      <parent link="${parent}"/>
+      <parent link="world"/>
       <child link="torso_base"/>
     </joint>

File: velma_description/robots/velma.urdf.xacro (robot description, xacro)
@@ -13,7 +13,15 @@
   <xacro:arg name="use_gazebo_kinect" default="false"/>
   <xacro:arg name="use_stereo_pair" default="false"/>
+  <xacro:arg name="mobile_base" default="false"/>
   <xacro:include filename="$(find lwr_defs)/defs/materials.xml"/>
   <xacro:include filename="$(find velma_description)/calibration/default_cal.xml"/>
-  <xacro:include filename="$(find velma_description)/defs/torso.urdf.xacro"/>
+  <xacro:if value="$(arg mobile_base)">
+    <xacro:include filename="$(find velma_description)/defs/torso_mobile.urdf.xacro"/>
+    <xacro:include filename="$(find velma_description)/defs/monokl.urdf.xacro"/>
+    <xacro:include filename="$(find velma_description)/defs/base_imu.urdf.xacro" />
+  </xacro:if>
+  <xacro:unless value="$(arg mobile_base)">
+    <xacro:include filename="$(find velma_description)/defs/torso.urdf.xacro"/>
+  </xacro:unless>
   <xacro:include filename="$(find velma_description)/defs/head.urdf.xacro" />
   <xacro:include filename="$(find lwr_defs)/defs/kuka_lwr_arm_defs.xml"/>
@@ -24,4 +32,5 @@
   <xacro:property name="camera_name" value="head_kinect" />
   <xacro:property name="stereo_name" value="head_stereo" />
+  <xacro:property name="M_PI" value="3.1415926535897931" />
   <!-- Gazebo Plugin -->
   <gazebo>
@@ -205,14 +214,78 @@
     </gazebo>
   </xacro:if>
-  <xacro:property name="M_PI" value="3.1415926535897931" />
-  <link name="world" />
-  <!-- static connection between the world frame and the map frame -->
-  <link name="map"/>
-  <joint name="world_map_joint" type="fixed">
-    <origin xyz="0 0 0" rpy="0 0 0"/>
-    <parent link="world"/>
-    <child link="map"/>
-  </joint>
-  <velma_torso parent="world" >
+  <xacro:if value="$(arg mobile_base)">
+    <gazebo reference="base_imu">
+      <selfCollide>true</selfCollide>
+      <sensor name="base_imu" type="imu">
+        <visualize>false</visualize>
+        <topic>/base_imu</topic>
+        <plugin name="base_imu" filename="libbase_imu.so" />
+        <imu>
+          <angular_velocity>
+            <x>
+              <noise type="gaussian">
+                <mean>0.0</mean>
+                <stddev>2e-4</stddev>
+                <bias_mean>0.0000075</bias_mean>
+                <bias_stddev>0.0000008</bias_stddev>
+              </noise>
+            </x>
+            <y>
+              <noise type="gaussian">
+                <mean>0.0</mean>
+                <stddev>2e-4</stddev>
+                <bias_mean>0.0000075</bias_mean>
+                <bias_stddev>0.0000008</bias_stddev>
+              </noise>
+            </y>
+            <z>
+              <noise type="gaussian">
+                <mean>0.0</mean>
+                <stddev>2e-4</stddev>
+                <bias_mean>0.0000075</bias_mean>
+                <bias_stddev>0.0000008</bias_stddev>
+              </noise>
+            </z>
+          </angular_velocity>
+          <linear_acceleration>
+            <x>
+              <noise type="gaussian">
+                <mean>0.0</mean>
+                <stddev>1.7e-2</stddev>
+                <bias_mean>0.1</bias_mean>
+                <bias_stddev>0.001</bias_stddev>
+              </noise>
+            </x>
+            <y>
+              <noise type="gaussian">
+                <mean>0.0</mean>
+                <stddev>1.7e-2</stddev>
+                <bias_mean>0.1</bias_mean>
+                <bias_stddev>0.001</bias_stddev>
+              </noise>
+            </y>
+            <z>
+              <noise type="gaussian">
+                <mean>0.0</mean>
+                <stddev>1.7e-2</stddev>
+                <bias_mean>0.1</bias_mean>
+                <bias_stddev>0.001</bias_stddev>
+              </noise>
+            </z>
+          </linear_acceleration>
+        </imu>
+      </sensor>
+    </gazebo>
+    <monokl name="monokl_l" parent="torso_base">
+      <origin xyz="0 0.3 0.256" rpy="0 0 0" />
+    </monokl>
+    <monokl name="monokl_r" parent="torso_base">
+      <origin xyz="0 -0.3 0.256" rpy="0 0 -${M_PI}" />
+    </monokl>
+    <base_imu name="base_imu" parent="torso_base">
+      <origin xyz="0 0 0.1225" rpy="0 0 0" />
+    </base_imu>
+  </xacro:if>
+  <velma_torso>
     <origin xyz="0 0 0" rpy="0 0 0"/>
   </velma_torso>

Commit message: added collision geometry for torso base

File: velma_description/defs/torso.urdf.xacro (robot description, xacro)
@@ -12,4 +12,5 @@
     </joint>
     <link name="torso_base">
+      <!--
       <visual>
         <origin xyz="0 0 0.1" rpy="0.0 0 0" />
@@ -21,4 +22,35 @@
         </material>
       </visual>
+    -->
+      <visual>
+        <origin xyz="0 0 0.1" rpy="0 0 0"/>
+        <geometry>
+          <box size="0.7 0.8 0.2" />
+        </geometry>
+        <material name="torso_base">
+          <color rgba="0.3 0.3 0.3 1"/>
+        </material>
+      </visual>
+      <visual>
+        <origin xyz="0 0 0.26" rpy="0 0 0"/>
+        <geometry>
+          <box size="0.4 0.4 0.12" />
+        </geometry>
+        <material name="torso_base">
+          <color rgba="0.3 0.3 0.3 1"/>
+        </material>
+      </visual>
+      <collision>
+        <origin xyz="0 0 0.1" rpy="0 0 0"/>
+        <geometry>
+          <box size="0.7 0.8 0.2" />
+        </geometry>
+      </collision>
+      <collision>
+        <origin xyz="0 0 0.26" rpy="0 0 0"/>
+        <geometry>
+          <box size="0.4 0.4 0.12" />
+        </geometry>
+      </collision>
 <!--
       <collision>

Commit message: allow self collisions of hands in some situations, added colors for Gazebo

File: velma_description/defs/torso.urdf.xacro (robot description, xacro)
@@ -78,4 +78,5 @@
       <turnGravityOff>false</turnGravityOff>
       <selfCollide>true</selfCollide>
+      <material>Gazebo/DarkGrey</material>
     </gazebo>
     <joint name="torso_0_joint" type="revolute">
@@ -153,4 +154,5 @@
       <turnGravityOff>false</turnGravityOff>
       <selfCollide>true</selfCollide>
+      <material>Gazebo/DarkGrey</material>
     </gazebo>
   </xacro:macro>

File: velma_description/robots/velma.urdf.xacro (robot description, xacro)
@@ -32,4 +32,26 @@
   <xacro:include filename="$(find velma_defs)/defs/kinect_camera.urdf.xacro" />
    -->
+  <xacro:macro name="visual_marker_xy" params="size pos_x pos_y pos_z">
+    <visual name="black_box1">
+      <origin xyz="${pos_x + 0.5*size} ${pos_y + 0.5*size} ${pos_z}" rpy="0 0 0" />
+      <geometry><box size="${size} ${size} 0.005" /></geometry>
+      <material name="Black" ><color rgba="0 0 0 1.0"/></material>
+    </visual>
+    <visual name="black_box2">
+      <origin xyz="${pos_x - 0.5*size} ${pos_y - 0.5*size} ${pos_z}" rpy="0 0 0" />
+      <geometry><box size="${size} ${size} 0.005" /></geometry>
+      <material name="Black" ><color rgba="0 0 0 1.0"/></material>
+    </visual>
+    <visual name="white_box1">
+      <origin xyz="${pos_x + 0.5*size} ${pos_y - 0.5*size} ${pos_z}" rpy="0 0 0" />
+      <geometry><box size="${size} ${size} 0.005" /></geometry>
+      <material name="White" ><color rgba="1 1 1 1.0"/></material>
+    </visual>
+    <visual name="white_box2">
+      <origin xyz="${pos_x - 0.5*size} ${pos_y + 0.5*size} ${pos_z}" rpy="0 0 0" />
+      <geometry><box size="${size} ${size} 0.005" /></geometry>
+      <material name="White" ><color rgba="1 1 1 1.0"/></material>
+    </visual>
+  </xacro:macro>
   <xacro:property name="camera_name" value="head_kinect" />
   <xacro:property name="stereo_name" value="head_stereo" />
@@ -347,4 +369,5 @@
       <inertia ixx="0.0007416" ixy="0" ixz="0.000566225" iyy="0.001365025" iyz="0" izz="0.0009347"/>
     </inertial>
+    <visual_marker_xy size="0.02" pos_x="0" pos_y="0" pos_z="0.05" />
   </link>
 <!--
@@ -401,4 +424,5 @@
       <inertia ixx="0.0007416" ixy="0" ixz="0.000566225" iyy="0.001365025" iyz="0" izz="0.0009347"/>
     </inertial>
+    <visual_marker_xy size="0.02" pos_x="0" pos_y="0" pos_z="0.02" />
   </link>
   <gazebo reference="left_gripper_mount_link">

Commit message: updated urdf model of velma

File: velma_description/defs/torso.urdf.xacro (robot description, xacro)
@@ -80,6 +80,11 @@
       <material>Gazebo/DarkGrey</material>
     </gazebo>
+    <!--
+      Changed joint origin from 0.1 to 0.03 (moved 7cm down) to make it similar to the real robot.
+      head_base - real height: 1.34
+      in urdf (with joint origin at 0.1): 1.41
+    -->
     <joint name="torso_0_joint" type="revolute">
-      <origin xyz="0 0 0.1" rpy="0 0 0"/>
+      <origin xyz="0 0 0.03" rpy="0 0 0"/>
       <axis xyz="0 0 1"/>
       <limit lower="-1.57" upper="1.57" effort="100" velocity="100"/>

Commit message: added big sphere as collision model for head

File: velma_description/defs/torso.urdf.xacro (robot description, xacro)
@@ -112,4 +112,10 @@
           </geometry>
         </collision>
+        <collision>
+          <origin xyz="0.04 0 1.57" rpy="0 0 0"/>
+          <geometry>
+            <sphere radius="0.24"/>
+          </geometry>
+        </collision>
       </xacro:if>
       <xacro:if value="${collision_detector == 'dart'}">
@@ -132,4 +138,10 @@
           </geometry>
         </collision>
+        <collision>
+          <origin xyz="0.04 0 1.57" rpy="0 0 0"/>
+          <geometry>
+            <sphere radius="0.24"/>
+          </geometry>
+        </collision>
       </xacro:if>
       <self_collision_checking>
@@ -143,4 +155,10 @@
         <geometry>
           <capsule radius="0.18" length="0.4"/>
+        </geometry>
+      </self_collision_checking>
+      <self_collision_checking>
+        <origin xyz="0.04 0 1.57" rpy="0 0 0"/>
+        <geometry>
+          <sphere radius="0.24"/>
         </geometry>
       </self_collision_checking>

Commit message: bugfix: octomap server

File: velma_description/defs/torso.urdf.xacro (robot description, xacro)
@@ -138,10 +138,4 @@
           </geometry>
         </collision>
-        <collision>
-          <origin xyz="0.04 0 1.57" rpy="0 0 0"/>
-          <geometry>
-            <sphere radius="0.24"/>
-          </geometry>
-        </collision>
       </xacro:if>
       <self_collision_checking>
@@ -157,10 +151,4 @@
         </geometry>
       </self_collision_checking>
-      <self_collision_checking>
-        <origin xyz="0.04 0 1.57" rpy="0 0 0"/>
-        <geometry>
-          <sphere radius="0.24"/>
-        </geometry>
-      </self_collision_checking>
       <inertial>
         <mass value="30.0"/>
@@ -174,4 +162,33 @@
       <material>Gazebo/DarkGrey</material>
     </gazebo>
+    <joint name="head_bounding_sphere_joint" type="fixed">
+      <origin xyz="0 0 0.03" rpy="0 0 0"/>
+      <parent link="torso_base"/>
+      <child link="head_bounding_sphere"/>
+    </joint>
+    <link name="head_bounding_sphere">
+      <collision>
+        <origin xyz="0.04 0 1.57" rpy="0 0 0"/>
+        <geometry>
+          <sphere radius="0.24"/>
+        </geometry>
+      </collision>
+      <self_collision_checking>
+        <origin xyz="0.04 0 1.57" rpy="0 0 0"/>
+        <geometry>
+          <sphere radius="0.24"/>
+        </geometry>
+      </self_collision_checking>
+      <inertial>
+        <mass value="0.3"/>
+        <origin rpy="0 0 0" xyz="0 -0.06 0.130"/>
+        <inertia ixx="0.03175" ixy="0" ixz="0" iyy="0.03175" iyz="0" izz="0.0135"/>
+      </inertial>
+    </link>
+    <gazebo reference="head_bounding_sphere">
+      <turnGravityOff>false</turnGravityOff>
+      <selfCollide>true</selfCollide>
+      <material>Gazebo/DarkGrey</material>
+    </gazebo>
   </xacro:macro>
 </robot>

Commit message: lower velocity limit for torso, added disabled collision pair for head-torso

File: velma_description/defs/torso.urdf.xacro (robot description, xacro)
@@ -90,5 +90,5 @@
       <origin xyz="0 0 0.03" rpy="0 0 0"/>
       <axis xyz="0 0 1"/>
-      <limit lower="-1.57" upper="1.57" effort="100" velocity="100"/>
+      <limit lower="-1.57" upper="1.57" effort="100" velocity="${30 * M_PI / 180}"/>
       <parent link="torso_base"/>
       <child link="torso_link0"/>
