Commit message: add calibration markers to robot model.

File: velma_description/robots/velma.urdf.xacro (robot description, xacro)
@@ -75,4 +75,18 @@
   <link name="right_gripper_calib_link">
   </link>
+  <joint name="right_gripper_calib_joint1" type="fixed">
+    <origin xyz="${cal_right_gripper_calib_link1_x} ${cal_right_gripper_calib_link1_y} ${cal_right_gripper_calib_link1_z}" rpy="${cal_right_gripper_calib_link1_roll} ${cal_right_gripper_calib_link1_pitch} ${cal_right_gripper_calib_link1_yaw}"/>
+    <parent link="right_arm_7_link"/>
+    <child link="right_gripper_calib_link1"/>
+  </joint>
+  <link name="right_gripper_calib_link1">
+  </link>
+  <joint name="right_gripper_calib_joint2" type="fixed">
+    <origin xyz="${cal_right_gripper_calib_link2_x} ${cal_right_gripper_calib_link2_y} ${cal_right_gripper_calib_link2_z}" rpy="${cal_right_gripper_calib_link2_roll} ${cal_right_gripper_calib_link2_pitch} ${cal_right_gripper_calib_link2_yaw}"/>
+    <parent link="right_arm_7_link"/>
+    <child link="right_gripper_calib_link2"/>
+  </joint>
+  <link name="right_gripper_calib_link2">
+  </link>
   <xacro:barret_hand prefix="left" parent="left_arm_7_link">
     <origin xyz="-0.115 0.0 -0.078" rpy="0 ${-M_PI/2} 0"/>
@@ -85,4 +99,18 @@
   <link name="left_gripper_calib_link">
   </link>
+  <joint name="left_gripper_calib_joint1" type="fixed">
+    <origin xyz="${cal_left_gripper_calib_link1_x} ${cal_left_gripper_calib_link1_y} ${cal_left_gripper_calib_link1_z}" rpy="${cal_left_gripper_calib_link1_roll} ${cal_left_gripper_calib_link1_pitch} ${cal_left_gripper_calib_link1_yaw}"/>
+    <parent link="left_arm_7_link"/>
+    <child link="left_gripper_calib_link1"/>
+  </joint>
+  <link name="left_gripper_calib_link1">
+  </link>
+  <joint name="left_gripper_calib_joint2" type="fixed">
+    <origin xyz="${cal_left_gripper_calib_link2_x} ${cal_left_gripper_calib_link2_y} ${cal_left_gripper_calib_link2_z}" rpy="${cal_left_gripper_calib_link2_roll} ${cal_left_gripper_calib_link2_pitch} ${cal_left_gripper_calib_link2_yaw}"/>
+    <parent link="left_arm_7_link"/>
+    <child link="left_gripper_calib_link2"/>
+  </joint>
+  <link name="left_gripper_calib_link2">
+  </link>
   <head_camera parent="left_arm_7_link" name="left_hand_camera">
       <origin xyz="${cal_left_hand_camera_joint_x} ${cal_left_hand_camera_joint_y} ${cal_left_hand_camera_joint_z}"

Commit message: added static map link to urdf

File: velma_description/robots/velma.urdf.xacro (robot description, xacro)
@@ -16,4 +16,11 @@
   <property name="M_PI" value="3.1415926535897931" />
   <link name="world" />
+  <!-- static connection between the world frame and the map frame -->
+  <link name="map" />
+  <joint name="world_map_joint" type="fixed">
+    <origin xyz="0 0 0" rpy="0 0 0"/>
+    <parent link="world"/>
+    <child link="map"/>
+  </joint>
   <velma_torso parent="world" >
     <origin xyz="0 0 0.1" rpy="0 0 0"/>

Commit message: options for collision model

File: velma_description/robots/velma.urdf.xacro (robot description, xacro)
@@ -5,4 +5,8 @@
                         xmlns:xacro="http://playerstage.sourceforge.net/gazebo/xmlschema/#interface"
 	 name="velma">
+  <xacro:arg name="collision_model_full" default="true"/>
+  <xacro:arg name="collision_model_simplified" default="false"/>
+  <xacro:arg name="collision_model_enlargement" default="0.0"/>
+  <xacro:arg name="collision_model_no_hands" default="false"/>
   <xacro:include filename="$(find velma_description)/calibration/default_cal.xml"/>
   <xacro:include filename="$(find velma_description)/defs/torso.urdf.xacro"/>
@@ -45,10 +49,12 @@
       <material name="Orange"/>
     </visual>
-    <collision>
-      <origin xyz="0 0 0" rpy="0 0 0"/>
-      <geometry>
-        <mesh filename="package://velma_description/meshes/collision/gripper_mount_collision.STL"/>
-      </geometry>
-    </collision>
+    <xacro:unless value="$(arg collision_model_no_hands)">
+      <collision>
+        <origin xyz="0 0 0" rpy="0 0 0"/>
+        <geometry>
+          <mesh filename="package://velma_description/meshes/collision/gripper_mount_collision.STL"/>
+        </geometry>
+      </collision>
+    </xacro:unless>
     <self_collision_checking>
       <origin xyz="0.05 0.0 -0.03" rpy="0 -0.81 0"/>
@@ -71,10 +77,12 @@
       <material name="Orange"/>
     </visual>
-    <collision>
-      <origin xyz="0 0 0" rpy="0 0 0"/>
-      <geometry>
-        <mesh filename="package://velma_description/meshes/collision/gripper_mount_collision.STL"/>
-      </geometry>
-    </collision>
+    <xacro:unless value="$(arg collision_model_no_hands)">
+      <collision>
+        <origin xyz="0 0 0" rpy="0 0 0"/>
+        <geometry>
+          <mesh filename="package://velma_description/meshes/collision/gripper_mount_collision.STL"/>
+        </geometry>
+      </collision>
+    </xacro:unless>
     <self_collision_checking>
       <origin xyz="0.05 0.0 -0.03" rpy="0 -0.81 0"/>

Commit message: better collision model

File: velma_description/robots/velma.urdf.xacro (robot description, xacro)
@@ -58,7 +58,7 @@
     </xacro:unless>
     <self_collision_checking>
-      <origin xyz="0.05 0.0 -0.03" rpy="0 -0.81 0"/>
+      <origin xyz="0.02 0.0 -0.03" rpy="0 ${M_PI/2.0} 0"/>
       <geometry>
-        <capsule radius="0.055" length="0.14"/>
+        <capsule radius="0.055" length="0.08"/>
       </geometry>
     </self_collision_checking>
@@ -86,7 +86,7 @@
     </xacro:unless>
     <self_collision_checking>
-      <origin xyz="0.05 0.0 -0.03" rpy="0 -0.81 0"/>
+      <origin xyz="0.02 0.0 -0.03" rpy="0 ${M_PI/2.0} 0"/>
       <geometry>
-        <capsule radius="0.055" length="0.14"/>
+        <capsule radius="0.055" length="0.08"/>
       </geometry>
     </self_collision_checking>

Commit message: collision model for ft sensor box

File: velma_description/robots/velma.urdf.xacro (robot description, xacro)
@@ -58,5 +58,5 @@
     </xacro:unless>
     <self_collision_checking>
-      <origin xyz="0.02 0.0 -0.03" rpy="0 ${M_PI/2.0} 0"/>
+      <origin xyz="0.02 0.0 0.0" rpy="0 ${M_PI/2.0} 0"/>
       <geometry>
         <capsule radius="0.055" length="0.08"/>

Commit message: ft tests

File: velma_description/robots/velma.urdf.xacro (robot description, xacro)
@@ -159,7 +159,7 @@
     </self_collision_checking>
     <inertial>
-      <mass value="0.2"/>
+      <mass value="0.002"/>
       <origin rpy="0 0 0" xyz="0 0 0.0625"/>
-      <inertia ixx="0.000520833333333" ixy="0" ixz="0" iyy="0.000520833333333" iyz="0" izz="0.000520833333333"/>
+      <inertia ixx="0.00000520833333333" ixy="0" ixz="0" iyy="0.00000520833333333" iyz="0" izz="0.00000520833333333"/>
     </inertial>
   </link>
@@ -195,7 +195,7 @@
     </self_collision_checking>
     <inertial>
-      <mass value="0.2"/>
+      <mass value="0.002"/>
       <origin rpy="0 0 0" xyz="0 0 0.0625"/>
-      <inertia ixx="0.000520833333333" ixy="0" ixz="0" iyy="0.000520833333333" iyz="0" izz="0.000520833333333"/>
+      <inertia ixx="0.00000520833333333" ixy="0" ixz="0" iyy="0.00000520833333333" iyz="0" izz="0.00000520833333333"/>
     </inertial>
   </link>

Commit message: added new joints for f/t sensors in gazebo

File: velma_description/robots/velma.urdf.xacro (robot description, xacro)
@@ -215,9 +215,57 @@
     <selfCollide>true</selfCollide>
   </gazebo>
-  <xacro:barret_hand prefix="right" parent="right_arm_7_link" with_optoforce="false">
+  <link name="right_FtSensorLink">
+    <inertial>
+      <mass value="0.002"/>
+      <origin rpy="0 0 0" xyz="0 0 0"/>
+      <inertia ixx="0.00000520833333333" ixy="0" ixz="0" iyy="0.00000520833333333" iyz="0" izz="0.00000520833333333"/>
+    </inertial>
+  </link>
+  <gazebo reference="right_FtSensorLink">
+    <turnGravityOff>false</turnGravityOff>
+    <selfCollide>false</selfCollide>
+  </gazebo>
+  <joint name="rightFtSensorJoint" type="revolute">
+    <parent link="right_gripper_mount_link"/>
+    <child link="right_FtSensorLink"/>
+                                  <!-- 39.56 degrees -->
     <origin xyz="0.115 0.0 -0.078" rpy="0 ${M_PI/2} 0"/>
+    <axis xyz="0 0 1"/>
+                          <!-- measured max angle is 94.  so upper limit is 94 - start orientation (42 degrees)-->
+    <limit effort="10" lower="0" upper="0" velocity="3.27"/>
+    <dynamics damping="0.05"/>
+  </joint>
+  <gazebo reference="rightFtSensorJoint">
+    <provideFeedback>true</provideFeedback>
+  </gazebo>
+  <xacro:barret_hand prefix="right" parent="right_FtSensorLink" with_optoforce="false">
+    <origin xyz="0 0 0" rpy="0 0 0"/>
   </xacro:barret_hand>
-  <xacro:barret_hand prefix="left" parent="left_arm_7_link" with_optoforce="true">
-    <origin xyz="-0.115 0.0 -0.078" rpy="0 ${-M_PI/2} 0"/>
+  <link name="left_FtSensorLink">
+    <inertial>
+      <mass value="0.002"/>
+      <origin rpy="0 0 0" xyz="0 0 0"/>
+      <inertia ixx="0.00000520833333333" ixy="0" ixz="0" iyy="0.00000520833333333" iyz="0" izz="0.00000520833333333"/>
+    </inertial>
+  </link>
+  <gazebo reference="left_FtSensorLink">
+    <turnGravityOff>false</turnGravityOff>
+    <selfCollide>false</selfCollide>
+  </gazebo>
+  <joint name="leftFtSensorJoint" type="revolute">
+    <parent link="left_gripper_mount_link"/>
+    <child link="left_FtSensorLink"/>
+                                  <!-- 39.56 degrees -->
+    <origin xyz="0.115 0.0 -0.078" rpy="0 ${M_PI/2} 0"/>
+    <axis xyz="0 0 1"/>
+                          <!-- measured max angle is 94.  so upper limit is 94 - start orientation (42 degrees)-->
+    <limit effort="10" lower="0" upper="0" velocity="3.27"/>
+    <dynamics damping="0.05"/>
+  </joint>
+  <gazebo reference="leftFtSensorJoint">
+    <provideFeedback>true</provideFeedback>
+  </gazebo>
+  <xacro:barret_hand prefix="left" parent="left_FtSensorLink" with_optoforce="true">
+    <origin xyz="0 0 0" rpy="0 0 ${M_PI}"/>
   </xacro:barret_hand>
 <!--

Commit message: more detailed gripper mount collision mesh

File: velma_description/robots/velma.urdf.xacro (robot description, xacro)
@@ -259,5 +259,5 @@
         <origin xyz="0 0 0" rpy="0 0 0"/>
         <geometry>
-          <mesh filename="package://velma_description/meshes/collision/gripper_mount_collision.STL"/>
+          <mesh filename="package://velma_description/meshes/collision/gripper_mount_collision2.STL"/>
         </geometry>
       </collision>
@@ -296,5 +296,5 @@
         <origin xyz="0 0 0" rpy="0 0 0"/>
         <geometry>
-          <mesh filename="package://velma_description/meshes/collision/gripper_mount_collision.STL"/>
+          <mesh filename="package://velma_description/meshes/collision/gripper_mount_collision2.STL"/>
         </geometry>
       </collision>

Commit message: updated collision model

File: velma_description/robots/velma.urdf.xacro (robot description, xacro)
@@ -270,7 +270,7 @@
     </self_collision_checking>
     <inertial>
-      <mass value="0.002"/>
+      <mass value="0.2"/>
       <origin rpy="0 0 0" xyz="0 0 0.0625"/>
-      <inertia ixx="0.00000520833333333" ixy="0" ixz="0" iyy="0.00000520833333333" iyz="0" izz="0.00000520833333333"/>
+      <inertia ixx="0.000520833333333" ixy="0" ixz="0" iyy="0.000520833333333" iyz="0" izz="0.000520833333333"/>
     </inertial>
   </link>
@@ -307,7 +307,7 @@
     </self_collision_checking>
     <inertial>
-      <mass value="0.002"/>
+      <mass value="0.2"/>
       <origin rpy="0 0 0" xyz="0 0 0.0625"/>
-      <inertia ixx="0.00000520833333333" ixy="0" ixz="0" iyy="0.00000520833333333" iyz="0" izz="0.00000520833333333"/>
+      <inertia ixx="0.000520833333333" ixy="0" ixz="0" iyy="0.000520833333333" iyz="0" izz="0.000520833333333"/>
     </inertial>
   </link>

Commit message: better inertia of gripper mount

File: velma_description/robots/velma.urdf.xacro (robot description, xacro)
@@ -270,9 +270,26 @@
     </self_collision_checking>
     <inertial>
-      <mass value="0.2"/>
-      <origin rpy="0 0 0" xyz="0 0 0.0625"/>
-      <inertia ixx="0.000520833333333" ixy="0" ixz="0" iyy="0.000520833333333" iyz="0" izz="0.000520833333333"/>
+      <mass value="0.2892125"/>
+      <origin rpy="0 0 0" xyz="0.0543534 0.0000315 -0.0313542"/>
+      <inertia ixx="0.0007416" ixy="0" ixz="0.000566225" iyy="0.001365025" iyz="0" izz="0.0009347"/>
     </inertial>
   </link>
+<!--
+gripper mount link:
+density: 1
+LOG: 2 Mesh Volume  is 0.000115685
+LOG: 2 Thin shell barycenter   0.546513   0.000319  -0.310379
+LOG: 2 Center of Mass  is 0.0543534 0.0000315 -0.0313542
+LOG: 2 Inertia Tensor is :
+LOG: 2     |  0.00000029664   0.00000000000   0.00000022649 |
+LOG: 2     |  0.00000000000   0.00000054601  -0.00000000000 |
+LOG: 2     |  0.00000022649  -0.00000000000   0.00000037388 |
+LOG: 2 Principal axes are :
+LOG: 2     |  0.764229   0.000001   0.644945 |
+LOG: 2     | -0.000000   1.000000  -0.000001 |
+LOG: 2     | -0.644945   0.000001   0.764229 |
+LOG: 2 axis momenta are :
+LOG: 2     |  0.010550   0.054601   0.056502 |
+-->
   <gazebo reference="right_gripper_mount_link">
     <turnGravityOff>false</turnGravityOff>
@@ -307,7 +324,7 @@
     </self_collision_checking>
     <inertial>
-      <mass value="0.2"/>
-      <origin rpy="0 0 0" xyz="0 0 0.0625"/>
-      <inertia ixx="0.000520833333333" ixy="0" ixz="0" iyy="0.000520833333333" iyz="0" izz="0.000520833333333"/>
+      <mass value="0.2892125"/>
+      <origin rpy="0 0 0" xyz="0.0543534 0.0000315 -0.0313542"/>
+      <inertia ixx="0.0007416" ixy="0" ixz="0.000566225" iyy="0.001365025" iyz="0" izz="0.0009347"/>
     </inertial>
   </link>

Commit message: collision model

File: velma_description/robots/velma.urdf.xacro (robot description, xacro)
@@ -271,5 +271,5 @@
     </xacro:unless>
     <self_collision_checking>
-      <origin xyz="0.02 0.0 0.0" rpy="0 ${M_PI/2.0} 0"/>
+      <origin xyz="0.02 0.0 0.01" rpy="0 ${M_PI/2.0} 0"/>
       <geometry>
         <capsule radius="0.055" length="0.08"/>
@@ -325,5 +325,5 @@
     </xacro:unless>
     <self_collision_checking>
-      <origin xyz="0.02 0.0 -0.03" rpy="0 ${M_PI/2.0} 0"/>
+      <origin xyz="0.02 0.0 -0.01" rpy="0 ${M_PI/2.0} 0"/>
       <geometry>
         <capsule radius="0.055" length="0.08"/>

Commit message: bugfix for wron mesh name in urdf

File: velma_description/robots/velma.urdf.xacro (robot description, xacro)
@@ -250,5 +250,5 @@
       <origin xyz="0 0 0" rpy="0.0 0 0" />
       <geometry>
-        <mesh filename="package://velma_description/meshes/gripper_mount_simplified.STL" />
+        <mesh filename="package://velma_description/meshes/gripper_mount_simplified.stl" />
       </geometry>
       <material name="Orange"/>
@@ -311,5 +311,5 @@
       <origin xyz="0 0 0" rpy="0.0 0 0" />
       <geometry>
-        <mesh filename="package://velma_description/meshes/gripper_mount_simplified.STL" />
+        <mesh filename="package://velma_description/meshes/gripper_mount_simplified.stl" />
       </geometry>
       <material name="Orange"/>

Commit message: higher kinect resolution, added stereo pair

File: velma_description/robots/velma.urdf.xacro (robot description, xacro)
@@ -9,15 +9,8 @@
   <xacro:arg name="collision_model_enlargement" default="0.0"/>
   <xacro:arg name="collision_model_no_hands" default="false"/>
-  <xacro:arg name="gazebo_scripts" default="false"/>
-  <xacro:arg name="gazebo_ops_file_re_body" default=""/>
-  <xacro:arg name="gazebo_ops_file_re_right_hand" default=""/>
-  <xacro:arg name="gazebo_ops_file_re_left_hand" default=""/>
-  <xacro:arg name="gazebo_ops_file_re_head" default=""/>
   <xacro:arg name="subsystem_xml" default="false"/>
   <xacro:arg name="xml_file_re_body" default=""/>
-  <xacro:arg name="xml_file_re_right_hand" default=""/>
-  <xacro:arg name="xml_file_re_left_hand" default=""/>
-  <xacro:arg name="xml_file_re_head" default=""/>
   <xacro:arg name="use_gazebo_kinect" default="false"/>
+  <xacro:arg name="use_stereo_pair" default="false"/>
   <xacro:include filename="$(find lwr_defs)/defs/materials.xml"/>
   <xacro:include filename="$(find velma_description)/calibration/default_cal.xml"/>
@@ -30,13 +23,9 @@
    -->
   <xacro:property name="camera_name" value="head_kinect" />
+  <xacro:property name="stereo_name" value="head_stereo" />
   <!-- Gazebo Plugin -->
   <gazebo>
     <plugin name="rtt_gazebo" filename="librtt_gazebo_deployer.so">
       <isolated/>
-      <xacro:if value="$(arg gazebo_scripts)">
-        <orocosScript>
-          <filename>$(arg gazebo_ops_file_re_body)</filename>
-        </orocosScript>
-      </xacro:if>
       <xacro:if value="$(arg subsystem_xml)">
         <subsystem_xml>
@@ -92,89 +81,5 @@
         <name>LeftHandOptoforce</name>
       </component>
-<!--
-      <component>
-        <package>velma_sim_gazebo</package>
-        <type>HeadGazebo</type>
-        <name>Head</name>
-      </component>
--->
     </plugin>
-<!--
-    <plugin name="rtt_gazebo" filename="librtt_gazebo_deployer.so">
-      <isolated/>
-      <xacro:if value="$(arg gazebo_scripts)">
-        <orocosScript>
-          <filename>$(arg gazebo_ops_file_re_right_hand)</filename>
-        </orocosScript>
-      </xacro:if>
-      <xacro:if value="$(arg subsystem_xml)">
-        <subsystem_xml>
-          <filename>$(arg xml_file_re_right_hand)</filename>
-        </subsystem_xml>
-      </xacro:if>
-      <master_service>
-        <name>velma_core_ve_hand</name>
-        <subname>right</subname>
-      </master_service>
-      <component>
-        <package>velma_sim_gazebo</package>
-        <type>BarrettHandGazebo</type>
-        <name>RightHand</name>
-      </component>
-      <component>
-        <package>velma_sim_gazebo</package>
-        <type>BarrettTactileGazebo</type>
-        <name>RightHandTactile</name>
-      </component>
-    </plugin>
-    <plugin name="rtt_gazebo" filename="librtt_gazebo_deployer.so">
-      <isolated/>
-      <xacro:if value="$(arg gazebo_scripts)">
-        <orocosScript>
-          <filename>$(arg gazebo_ops_file_re_left_hand)</filename>
-        </orocosScript>
-      </xacro:if>
-      <xacro:if value="$(arg subsystem_xml)">
-        <subsystem_xml>
-          <filename>$(arg xml_file_re_left_hand)</filename>
-        </subsystem_xml>
-      </xacro:if>
-      <master_service>
-        <name>velma_core_ve_hand</name>
-        <subname>left</subname>
-      </master_service>
-      <component>
-        <package>velma_sim_gazebo</package>
-        <type>BarrettHandGazebo</type>
-        <name>LeftHand</name>
-      </component>
-      <component>
-        <package>velma_sim_gazebo</package>
-        <type>OptoforceGazebo</type>
-        <name>LeftHandOptoforce</name>
-      </component>
-    </plugin>
-    <plugin name="rtt_gazebo" filename="librtt_gazebo_deployer.so">
-      <isolated/>
-      <xacro:if value="$(arg gazebo_scripts)">
-        <orocosScript>
-          <filename>$(arg gazebo_ops_file_re_head)</filename>
-        </orocosScript>
-      </xacro:if>
-      <xacro:if value="$(arg subsystem_xml)">
-        <subsystem_xml>
-          <filename>$(arg xml_file_re_head)</filename>
-        </subsystem_xml>
-      </xacro:if>
-      <master_service>
-        <name>velma_core_ve_head</name>
-      </master_service>
-      <component>
-        <package>velma_sim_gazebo</package>
-        <type>HeadGazebo</type>
-        <name>Head</name>
-      </component>
-    </plugin>
--->
   </gazebo>
   <xacro:if value="$(arg use_gazebo_kinect)">
@@ -187,6 +92,6 @@
           <horizontal_fov>1.047</horizontal_fov>
           <image>
-            <width>400</width>
-            <height>300</height>
+            <width>800</width>
+            <height>600</height>
             <format>B8G8R8</format>
           </image>
@@ -209,4 +114,80 @@
           <pointCloudCutoff>0.5</pointCloudCutoff>
           <pointCloudCutoffMax>3.0</pointCloudCutoffMax>
+          <distortionK1>0.00000001</distortionK1>
+          <distortionK2>0.00000001</distortionK2>
+          <distortionK3>0.00000001</distortionK3>
+          <distortionT1>0.00000001</distortionT1>
+          <distortionT2>0.00000001</distortionT2>
+          <CxPrime>0</CxPrime>
+          <Cx>0</Cx>
+          <Cy>0</Cy>
+          <focalLength>0</focalLength>
+          <hackBaseline>0</hackBaseline>
+        </plugin>
+      </sensor>
+    </gazebo>
+  </xacro:if>
+  <xacro:if value="$(arg use_stereo_pair)">
+    <gazebo reference="stereo_left_link">
+      <sensor type="camera" name="stereo_left_camera">
+        <always_on>0</always_on>
+        <update_rate>15.0</update_rate>
+        <visualize>false</visualize>
+        <camera>
+          <horizontal_fov>1.047</horizontal_fov>
+          <image>
+            <width>400</width>
+            <height>300</height>
+            <format>B8G8R8</format>
+          </image>
+          <clip>
+            <near>0.1</near>
+            <far>10</far>
+          </clip>
+        </camera>
+        <plugin name="camera_left_controller" filename="libgazebo_ros_camera.so">
+          <baseline>0.2</baseline>
+          <cameraName>${stereo_name}_left</cameraName>
+          <imageTopicName>/${stereo_name}_left/image_raw</imageTopicName>
+          <cameraInfoTopicName>/${stereo_name}_left/camera_info</cameraInfoTopicName>
+          <frameName>stereo_left_optical_frame</frameName>
+          <updateRate>15</updateRate>
+          <distortionK1>0.00000001</distortionK1>
+          <distortionK2>0.00000001</distortionK2>
+          <distortionK3>0.00000001</distortionK3>
+          <distortionT1>0.00000001</distortionT1>
+          <distortionT2>0.00000001</distortionT2>
+          <CxPrime>0</CxPrime>
+          <Cx>0</Cx>
+          <Cy>0</Cy>
+          <focalLength>0</focalLength>
+          <hackBaseline>0</hackBaseline>
+        </plugin>
+      </sensor>
+    </gazebo>
+    <gazebo reference="stereo_right_link">
+      <sensor type="camera" name="stereo_right_camera">
+        <always_on>0</always_on>
+        <update_rate>15.0</update_rate>
+        <visualize>false</visualize>
+        <camera>
+          <horizontal_fov>1.047</horizontal_fov>
+          <image>
+            <width>400</width>
+            <height>300</height>
+            <format>B8G8R8</format>
+          </image>
+          <clip>
+            <near>0.1</near>
+            <far>10</far>
+          </clip>
+        </camera>
+        <plugin name="camera_right_controller" filename="libgazebo_ros_camera.so">
+          <baseline>0.2</baseline>
+          <cameraName>${stereo_name}_right</cameraName>
+          <imageTopicName>/${stereo_name}_right/image_raw</imageTopicName>
+          <cameraInfoTopicName>/${stereo_name}_right/camera_info</cameraInfoTopicName>
+          <frameName>stereo_right_optical_frame</frameName>
+          <updateRate>15</updateRate>
           <distortionK1>0.00000001</distortionK1>
           <distortionK2>0.00000001</distortionK2>
