Commit message: set limits in sensor joint to admissible values

File: velma_description/robots/velma.urdf.xacro (robot description, xacro)
@@ -338,5 +338,5 @@
     <axis xyz="0 0 1"/>
                           <!-- measured max angle is 94.  so upper limit is 94 - start orientation (42 degrees)-->
-    <limit effort="10" lower="0" upper="0" velocity="3.27"/>
+    <limit effort="10" lower="0" upper="0.00001" velocity="3.27"/>
     <dynamics damping="0.05"/>
   </joint>
@@ -365,5 +365,5 @@
     <axis xyz="0 0 1"/>
                           <!-- measured max angle is 94.  so upper limit is 94 - start orientation (42 degrees)-->
-    <limit effort="10" lower="0" upper="0" velocity="3.27"/>
+    <limit effort="10" lower="0" upper="0.00001" velocity="3.27"/>
     <dynamics damping="0.05"/>
   </joint>

Commit message: added virtual link ee_link

File: velma_description/robots/velma.urdf.xacro (robot description, xacro)
@@ -343,5 +343,5 @@
   <joint name="right_gripper_mount_joint" type="fixed">
     <origin xyz="0 0 0" rpy="0 0 0"/>
-    <parent link="right_arm_7_link"/>
+    <parent link="right_arm_ee_link"/>
     <child link="right_gripper_mount_link"/>
   </joint>
@@ -405,5 +405,5 @@
   <joint name="left_gripper_mount_joint" type="fixed">
     <origin xyz="0 0 0" rpy="0 0 ${M_PI}"/>
-    <parent link="left_arm_7_link"/>
+    <parent link="left_arm_ee_link"/>
     <child link="left_gripper_mount_link"/>
   </joint>

Commit message: added 0,5cm offset of BH base

File: velma_description/robots/velma.urdf.xacro (robot description, xacro)
@@ -466,5 +466,5 @@
   </gazebo>
   <xacro:barret_hand prefix="right" parent="right_FtSensorLink" with_optoforce="$(arg use_right_optoforces)">
-    <origin xyz="0 0 0" rpy="0 0 0"/>
+    <origin xyz="0 0 0.005" rpy="0 0 0"/>
   </xacro:barret_hand>
   <link name="left_FtSensorLink">
@@ -493,5 +493,5 @@
   </gazebo>
   <xacro:barret_hand prefix="left" parent="left_FtSensorLink" with_optoforce="$(arg use_left_optoforces)">
-    <origin xyz="0 0 0" rpy="0 0 ${M_PI}"/>
+    <origin xyz="0 0 0.005" rpy="0 0 ${M_PI}"/>
   </xacro:barret_hand>
 <!--

Commit message: added tools for calibration

File: velma_description/robots/velma.urdf.xacro (robot description, xacro)
@@ -407,4 +407,18 @@
     <visual_marker_xy size="0.02" pos_x="0" pos_y="0" pos_z="0.05" />
   </link>
+  <joint name="right_gripper_mount_joint" type="fixed">
+    <origin xyz="0 0 0.112" rpy="0 0 0"/>
+    <parent link="right_arm_ee_link"/>
+    <child link="right_needle_link"/>
+  </joint>
+  <link name="right_needle_link">
+  </link>
+  <joint name="left_gripper_mount_joint" type="fixed">
+    <origin xyz="0 0 0.109" rpy="0 0 0"/>
+    <parent link="left_arm_ee_link"/>
+    <child link="left_needle_link"/>
+  </joint>
+  <link name="left_needle_link">
+  </link>
 <!--
 gripper mount link:

Commit message: added tools for calibration

File: velma_description/robots/velma.urdf.xacro (robot description, xacro)
@@ -407,5 +407,5 @@
     <visual_marker_xy size="0.02" pos_x="0" pos_y="0" pos_z="0.05" />
   </link>
-  <joint name="right_gripper_mount_joint" type="fixed">
+  <joint name="right_needle_joint" type="fixed">
     <origin xyz="0 0 0.112" rpy="0 0 0"/>
     <parent link="right_arm_ee_link"/>
@@ -414,5 +414,5 @@
   <link name="right_needle_link">
   </link>
-  <joint name="left_gripper_mount_joint" type="fixed">
+  <joint name="left_needle_joint" type="fixed">
     <origin xyz="0 0 0.109" rpy="0 0 0"/>
     <parent link="left_arm_ee_link"/>

Commit message: new calibration

File: velma_description/robots/velma.urdf.xacro (robot description, xacro)
@@ -339,5 +339,5 @@
   </velma_torso>
   <kuka_lwr_arm parent="torso_link0" name="right" right="1">
-    <origin xyz="0 -0.000188676 1.17335" rpy="0 ${-M_PI/3} ${M_PI/2}"/>
+    <origin xyz="${cal_torso_link2_right_arm_base_joint_x} ${cal_torso_link2_right_arm_base_joint_y} ${cal_torso_link2_right_arm_base_joint_z}" rpy="${cal_torso_link2_right_arm_base_joint_roll} ${cal_torso_link2_right_arm_base_joint_pitch} ${cal_torso_link2_right_arm_base_joint_yaw}"/>
   </kuka_lwr_arm>
   <kuka_lwr_arm parent="torso_link0" name="left" right="1">
@@ -408,5 +408,5 @@
   </link>
   <joint name="right_needle_joint" type="fixed">
-    <origin xyz="0 0 0.112" rpy="0 0 0"/>
+    <origin xyz="${cal_right_needle_joint_x} ${cal_right_needle_joint_y} ${cal_right_needle_joint_z}" rpy="0 0 0"/>
     <parent link="right_arm_ee_link"/>
     <child link="right_needle_link"/>
@@ -415,5 +415,5 @@
   </link>
   <joint name="left_needle_joint" type="fixed">
-    <origin xyz="0 0 0.109" rpy="0 0 0"/>
+    <origin xyz="${cal_left_needle_joint_x} ${cal_left_needle_joint_y} ${cal_left_needle_joint_z}" rpy="0 0 0"/>
     <parent link="left_arm_ee_link"/>
     <child link="left_needle_link"/>

Commit message: added needle collision element to urdf

File: velma_description/robots/velma.urdf.xacro (robot description, xacro)
@@ -394,4 +394,11 @@
       </xacro:if>
     </xacro:unless>
+    <!-- needle -->
+    <collision>
+      <origin xyz="0 0 0.07" rpy="0 0 0"/>
+      <geometry>
+        <box size="0.05 0.05 0.14"/>
+      </geometry>
+    </collision>
     <self_collision_checking>
       <origin xyz="0.02 0.0 0.01" rpy="0 ${M_PI/2.0} 0"/>
@@ -485,4 +492,11 @@
       </xacro:if>
     </xacro:unless>
+    <!-- needle -->
+    <collision>
+      <origin xyz="0 0 0.07" rpy="0 0 0"/>
+      <geometry>
+        <box size="0.05 0.05 0.14"/>
+      </geometry>
+    </collision>
     <self_collision_checking>
       <origin xyz="0.02 0.0 -0.01" rpy="0 ${M_PI/2.0} 0"/>

Commit message: added 0 mass param for dummy links

File: velma_description/robots/velma.urdf.xacro (robot description, xacro)
@@ -420,4 +420,9 @@
   </joint>
   <link name="right_needle_link">
+    <inertial>
+      <mass value="0"/>
+      <origin rpy="0 0 0" xyz="0 0 0"/>
+      <inertia ixx="0" ixy="0" ixz="0" iyy="0" iyz="0" izz="0"/>
+    </inertial>
   </link>
   <joint name="left_needle_joint" type="fixed">
@@ -427,4 +432,9 @@
   </joint>
   <link name="left_needle_link">
+    <inertial>
+      <mass value="0"/>
+      <origin rpy="0 0 0" xyz="0 0 0"/>
+      <inertia ixx="0" ixy="0" ixz="0" iyy="0" iyz="0" izz="0"/>
+    </inertial>
   </link>
 <!--

Commit message: added collision models for additional >needle< tool

File: velma_description/robots/velma.urdf.xacro (robot description, xacro)
@@ -402,4 +402,10 @@
     </collision>
     <self_collision_checking>
+      <origin xyz="0 0 0.07" rpy="0 0 0"/>
+      <geometry>
+        <capsule radius="0.025" length="0.09"/>
+      </geometry>
+    </self_collision_checking>
+    <self_collision_checking>
       <origin xyz="0.02 0.0 0.01" rpy="0 ${M_PI/2.0} 0"/>
       <geometry>
@@ -510,4 +516,10 @@
     </collision>
     <self_collision_checking>
+      <origin xyz="0 0 0.07" rpy="0 0 0"/>
+      <geometry>
+        <capsule radius="0.025" length="0.09"/>
+      </geometry>
+    </self_collision_checking>
+    <self_collision_checking>
       <origin xyz="0.02 0.0 -0.01" rpy="0 ${M_PI/2.0} 0"/>
       <geometry>

Commit message: added virtual links for orientation constraints

File: velma_description/robots/velma.urdf.xacro (robot description, xacro)
@@ -636,3 +636,81 @@
     <origin xyz="${cal_head_base_joint_x} ${cal_head_base_joint_y} ${cal_head_base_joint_z}" rpy="${cal_head_base_joint_roll} ${cal_head_base_joint_pitch} ${cal_head_base_joint_yaw}"/>
   </xacro:velma_head>
+  <!-- This is a part of the tree that is used to enable orientation constraints
+       for the end-effectors in planning. -->
+  <joint name="rightKeepUprightJoint0" type="revolute">
+    <parent link="right_arm_ee_link"/>
+    <child link="right_keepUprightLink1"/>
+    <origin xyz="0 0 0" rpy="0 0 0"/>
+    <axis xyz="0 0 1"/>
+    <limit effort="10" lower="${-M_PI}" upper="${M_PI}" velocity="3.27"/>
+    <dynamics damping="0.05"/>
+  </joint>
+  <link name="right_keepUprightLink1">
+    <inertial>
+      <mass value="0.002"/>
+      <origin rpy="0 0 0" xyz="0 0 0"/>
+      <inertia ixx="0.00000520833333333" ixy="0" ixz="0" iyy="0.00000520833333333" iyz="0" izz="0.00000520833333333"/>
+    </inertial>
+  </link>
+  <gazebo reference="right_keepUprightLink1">
+    <turnGravityOff>false</turnGravityOff>
+    <selfCollide>true</selfCollide>
+  </gazebo>
+  <joint name="rightKeepUprightJoint1" type="revolute">
+    <parent link="right_keepUprightLink1"/>
+    <child link="right_keepUprightLink2"/>
+    <origin xyz="0 0 0" rpy="0 ${M_PI/2} 0"/>
+    <axis xyz="0 0 1"/>
+    <limit effort="10" lower="${-M_PI}" upper="${M_PI}" velocity="3.27"/>
+    <dynamics damping="0.05"/>
+  </joint>
+  <link name="right_keepUprightLink2">
+    <inertial>
+      <mass value="0.002"/>
+      <origin rpy="0 0 0" xyz="0 0 0"/>
+      <inertia ixx="0.00000520833333333" ixy="0" ixz="0" iyy="0.00000520833333333" iyz="0" izz="0.00000520833333333"/>
+    </inertial>
+  </link>
+  <gazebo reference="right_keepUprightLink2">
+    <turnGravityOff>false</turnGravityOff>
+    <selfCollide>true</selfCollide>
+  </gazebo>
+  <joint name="leftKeepUprightJoint0" type="revolute">
+    <parent link="left_arm_ee_link"/>
+    <child link="left_keepUprightLink1"/>
+    <origin xyz="0 0 0" rpy="0 0 0"/>
+    <axis xyz="0 0 1"/>
+    <limit effort="10" lower="${-M_PI}" upper="${M_PI}" velocity="3.27"/>
+    <dynamics damping="0.05"/>
+  </joint>
+  <link name="left_keepUprightLink1">
+    <inertial>
+      <mass value="0.002"/>
+      <origin rpy="0 0 0" xyz="0 0 0"/>
+      <inertia ixx="0.00000520833333333" ixy="0" ixz="0" iyy="0.00000520833333333" iyz="0" izz="0.00000520833333333"/>
+    </inertial>
+  </link>
+  <gazebo reference="left_keepUprightLink1">
+    <turnGravityOff>false</turnGravityOff>
+    <selfCollide>true</selfCollide>
+  </gazebo>
+  <joint name="leftKeepUprightJoint1" type="revolute">
+    <parent link="left_keepUprightLink1"/>
+    <child link="left_keepUprightLink2"/>
+    <origin xyz="0 0 0" rpy="0 ${M_PI/2} 0"/>
+    <axis xyz="0 0 1"/>
+    <limit effort="10" lower="${-M_PI}" upper="${M_PI}" velocity="3.27"/>
+    <dynamics damping="0.05"/>
+  </joint>
+  <link name="left_keepUprightLink2">
+    <inertial>
+      <mass value="0.002"/>
+      <origin rpy="0 0 0" xyz="0 0 0"/>
+      <inertia ixx="0.00000520833333333" ixy="0" ixz="0" iyy="0.00000520833333333" iyz="0" izz="0.00000520833333333"/>
+    </inertial>
+  </link>
+  <gazebo reference="left_keepUprightLink2">
+    <turnGravityOff>false</turnGravityOff>
+    <selfCollide>true</selfCollide>
+  </gazebo>
 </robot>

Commit message: added calibration needles as optional feature in urdf

File: velma_description/robots/velma.urdf.xacro (robot description, xacro)
@@ -19,4 +19,5 @@
   <xacro:arg name="use_right_optoforces" default="false"/>
   <xacro:arg name="use_dh_compatible_model" default="false"/>
+  <xacro:arg name="calibration_needles" default="false"/>
   <xacro:include filename="$(find lwr_defs)/defs/materials.xml"/>
   <xacro:include filename="$(find velma_description)/calibration/default_cal.xml"/>
@@ -391,17 +392,19 @@
       </xacro:if>
     </xacro:unless>
-    <!-- needle -->
-    <collision>
-      <origin xyz="0 0 0.07" rpy="0 0 0"/>
-      <geometry>
-        <box size="0.05 0.05 0.14"/>
-      </geometry>
-    </collision>
-    <self_collision_checking>
-      <origin xyz="0 0 0.07" rpy="0 0 0"/>
-      <geometry>
-        <capsule radius="0.025" length="0.09"/>
-      </geometry>
-    </self_collision_checking>
+    <xacro:if value="$(arg calibration_needles)">
+      <!-- needle -->
+      <collision>
+        <origin xyz="0 0 0.07" rpy="0 0 0"/>
+        <geometry>
+          <box size="0.05 0.05 0.14"/>
+        </geometry>
+      </collision>
+      <self_collision_checking>
+        <origin xyz="0 0 0.07" rpy="0 0 0"/>
+        <geometry>
+          <capsule radius="0.025" length="0.09"/>
+        </geometry>
+      </self_collision_checking>
+    </xacro:if>
     <self_collision_checking>
       <origin xyz="0.02 0.0 0.01" rpy="0 ${M_PI/2.0} 0"/>
@@ -417,28 +420,30 @@
     <xacro:visual_marker_xy size="0.02" pos_x="0" pos_y="0" pos_z="0.05" />
   </link>
-  <joint name="right_needle_joint" type="fixed">
-    <origin xyz="${cal_right_needle_joint_x} ${cal_right_needle_joint_y} ${cal_right_needle_joint_z}" rpy="0 0 0"/>
-    <parent link="right_arm_ee_link"/>
-    <child link="right_needle_link"/>
-  </joint>
-  <link name="right_needle_link">
-    <inertial>
-      <mass value="0"/>
-      <origin rpy="0 0 0" xyz="0 0 0"/>
-      <inertia ixx="0" ixy="0" ixz="0" iyy="0" iyz="0" izz="0"/>
-    </inertial>
-  </link>
-  <joint name="left_needle_joint" type="fixed">
-    <origin xyz="${cal_left_needle_joint_x} ${cal_left_needle_joint_y} ${cal_left_needle_joint_z}" rpy="0 0 0"/>
-    <parent link="left_arm_ee_link"/>
-    <child link="left_needle_link"/>
-  </joint>
-  <link name="left_needle_link">
-    <inertial>
-      <mass value="0"/>
-      <origin rpy="0 0 0" xyz="0 0 0"/>
-      <inertia ixx="0" ixy="0" ixz="0" iyy="0" iyz="0" izz="0"/>
-    </inertial>
-  </link>
+  <xacro:if value="$(arg calibration_needles)">
+    <joint name="right_needle_joint" type="fixed">
+      <origin xyz="${cal_right_needle_joint_x} ${cal_right_needle_joint_y} ${cal_right_needle_joint_z}" rpy="0 0 0"/>
+      <parent link="right_arm_ee_link"/>
+      <child link="right_needle_link"/>
+    </joint>
+    <link name="right_needle_link">
+      <inertial>
+        <mass value="0"/>
+        <origin rpy="0 0 0" xyz="0 0 0"/>
+        <inertia ixx="0" ixy="0" ixz="0" iyy="0" iyz="0" izz="0"/>
+      </inertial>
+    </link>
+    <joint name="left_needle_joint" type="fixed">
+      <origin xyz="${cal_left_needle_joint_x} ${cal_left_needle_joint_y} ${cal_left_needle_joint_z}" rpy="0 0 0"/>
+      <parent link="left_arm_ee_link"/>
+      <child link="left_needle_link"/>
+    </joint>
+    <link name="left_needle_link">
+      <inertial>
+        <mass value="0"/>
+        <origin rpy="0 0 0" xyz="0 0 0"/>
+        <inertia ixx="0" ixy="0" ixz="0" iyy="0" iyz="0" izz="0"/>
+      </inertial>
+    </link>
+  </xacro:if>
 <!--
 gripper mount link:
@@ -505,17 +510,19 @@
       </xacro:if>
     </xacro:unless>
-    <!-- needle -->
-    <collision>
-      <origin xyz="0 0 0.07" rpy="0 0 0"/>
-      <geometry>
-        <box size="0.05 0.05 0.14"/>
-      </geometry>
-    </collision>
-    <self_collision_checking>
-      <origin xyz="0 0 0.07" rpy="0 0 0"/>
-      <geometry>
-        <capsule radius="0.025" length="0.09"/>
-      </geometry>
-    </self_collision_checking>
+    <xacro:if value="$(arg calibration_needles)">
+      <!-- needle -->
+      <collision>
+        <origin xyz="0 0 0.07" rpy="0 0 0"/>
+        <geometry>
+          <box size="0.05 0.05 0.14"/>
+        </geometry>
+      </collision>
+      <self_collision_checking>
+        <origin xyz="0 0 0.07" rpy="0 0 0"/>
+        <geometry>
+          <capsule radius="0.025" length="0.09"/>
+        </geometry>
+      </self_collision_checking>
+    </xacro:if>
     <self_collision_checking>
       <origin xyz="0.02 0.0 -0.01" rpy="0 ${M_PI/2.0} 0"/>

Commit message: changed colors of some visuals

File: velma_description/robots/velma.urdf.xacro (robot description, xacro)
@@ -353,5 +353,7 @@
         <mesh filename="package://velma_description/meshes/gripper_mount_simplified.stl" />
       </geometry>
-      <material name="Orange"/>
+        <material name="Orange" >
+          <color rgba="1 0.5 0 1.0"/>
+        </material>
     </visual>
     <visual>
@@ -360,5 +362,7 @@
         <mesh filename="package://velma_description/meshes/imu_case_right.stl" />
       </geometry>
-      <material name="Orange"/>
+        <material name="Orange" >
+          <color rgba="1 0.5 0 1.0"/>
+        </material>
     </visual>
     <xacro:unless value="$(arg collision_model_no_hands)">
@@ -478,5 +482,7 @@
         <mesh filename="package://velma_description/meshes/gripper_mount_simplified.stl" />
       </geometry>
-      <material name="Orange"/>
+        <material name="Orange" >
+          <color rgba="1 0.5 0 1.0"/>
+        </material>
     </visual>
     <xacro:unless value="$(arg collision_model_no_hands)">
