Commit message: cleanup

File: velma_description/urdf/head/head.urdf.xacro (robot description, xacro)
@@ -203,4 +203,10 @@
       <turnGravityOff>false</turnGravityOff>
       <selfCollide>true</selfCollide>
+       <material>Gazebo/DarkGrey</material>
+    </gazebo>
+    <gazebo reference="head_tilt_link_dummy">
+      <turnGravityOff>false</turnGravityOff>
+      <selfCollide>true</selfCollide>
+       <material>Gazebo/DarkGrey</material>
     </gazebo>
     <!-- sensors -->

File: velma_description/urdf/torso/torso.urdf.xacro (robot description, xacro)
@@ -31,5 +31,5 @@
         </geometry>
         <material name="torso_base">
-          <color rgba="0.3 0.3 0.3 1"/>
+          <color rgba="0.4 0.4 0.4 1"/>
         </material>
       </visual>
@@ -40,5 +40,5 @@
         </geometry>
         <material name="torso_base">
-          <color rgba="0.3 0.3 0.3 1"/>
+          <color rgba="0.4 0.4 0.4 1"/>
         </material>
       </visual>
@@ -80,5 +80,8 @@
       <turnGravityOff>false</turnGravityOff>
       <selfCollide>true</selfCollide>
-      <material>Gazebo/DarkGrey</material>
+      <material>
+          <diffuse>0.4 0.4 0.4 1</diffuse>
+          <ambient>0.4 0.4 0.4 1</ambient>
+      </material>
     </gazebo>
     <!--

File: velma_description/urdf/velma.urdf.xacro (robot description, xacro)
@@ -5,4 +5,7 @@
                         xmlns:xacro="http://www.ros.org/wiki/xacro"
 	 name="velma">
+  <gazebo>
+    <selfCollide>true</selfCollide>
+  </gazebo>
   <xacro:arg name="collision_model_full" default="false"/>
   <xacro:arg name="collision_model_simplified" default="true"/>
@@ -69,74 +72,4 @@
   <xacro:property name="M_PI" value="3.1415926535897931" />
   <!-- Gazebo Plugin -->
-  <gazebo>
-    <plugin name="rtt_gazebo" filename="librtt_gazebo_deployer.so">
-      <isolated/>
-      <collision_detector>${collision_detector}</collision_detector>
-      <xacro:if value="$(arg subsystem_xml)">
-        <subsystem_xml>
-          <filename>$(arg xml_file_re_body)</filename>
-        </subsystem_xml>
-      </xacro:if>
-      <master_service>
-        <name>velma_sim_gazebo</name>
-        <subname>velma_sim_gazebo</subname>
-      </master_service>
-      <component>
-        <package>velma_sim_gazebo</package>
-        <type>TorsoGazebo</type>
-        <name>TorsoSim</name>
-      </component>
-      <component>
-        <package>velma_sim_gazebo</package>
-        <type>LWRGazebo</type>
-        <name>LWRrSim</name>
-      </component>
-      <component>
-        <package>velma_sim_gazebo</package>
-        <type>LWRGazebo</type>
-        <name>LWRlSim</name>
-      </component>
-      <component>
-        <package>velma_sim_gazebo</package>
-        <type>FtSensorGazebo</type>
-        <name>LeftFtSensor</name>
-      </component>
-      <component>
-        <package>velma_sim_gazebo</package>
-        <type>FtSensorGazebo</type>
-        <name>RightFtSensor</name>
-      </component>
-      <component>
-        <package>velma_sim_gazebo</package>
-        <type>BarrettHandGazebo</type>
-        <name>RightHand</name>
-      </component>
-      <component>
-        <package>velma_sim_gazebo</package>
-        <type>BarrettTactileGazebo</type>
-        <name>RightHandTactile</name>
-      </component>
-      <component>
-        <package>velma_sim_gazebo</package>
-        <type>OptoforceGazebo</type>
-        <name>RightHandOptoforce</name>
-      </component>
-      <component>
-        <package>velma_sim_gazebo</package>
-        <type>BarrettHandGazebo</type>
-        <name>LeftHand</name>
-      </component>
-      <component>
-        <package>velma_sim_gazebo</package>
-        <type>BarrettTactileGazebo</type>
-        <name>LeftHandTactile</name>
-      </component>
-      <component>
-        <package>velma_sim_gazebo</package>
-        <type>OptoforceGazebo</type>
-        <name>LeftHandOptoforce</name>
-      </component>
-    </plugin>
-  </gazebo>
   <xacro:if value="$(arg use_gazebo_kinect)">
     <gazebo reference="head_kinect_rgb_link">
@@ -727,31 +660,3 @@
     <selfCollide>true</selfCollide>
   </gazebo>
-  <!-- Floating gripper -->
-  <xacro:include filename="hand/floating_gripper_joint.xacro"/>
-  <xacro:floating_gripper_joint parent="world" />
-<!--   <link name="floating_FtSensorLink">
-    <inertial>
-      <mass value="0.002"/>
-      <origin rpy="0 0 0" xyz="0 0 0"/>
-      <inertia ixx="0.00000520833333333" ixy="0" ixz="0" iyy="0.00000520833333333" iyz="0" izz="0.00000520833333333"/>
-    </inertial>
-  </link>
-  <joint name="floatingFtSensorJoint" type="revolute">
-    <parent link="floating_gripper_mount_link"/>
-    <child link="floating_FtSensorLink"/>
-    <origin xyz="0.115 0.0 -0.078" rpy="0 ${M_PI/2} 0"/>
-    <axis xyz="0 0 1"/>
-    <limit effort="10" lower="0" upper="${M_PI}" velocity="3.27"/>
-    <dynamics damping="0.05"/>
-  </joint>
-  <gazebo reference="leftFtSensorJoint">
-    <provideFeedback>true</provideFeedback>
-  </gazebo>
-  <xacro:barret_hand prefix="left" parent="left_FtSensorLink" with_optoforce="$(arg use_left_optoforces)">
-    <origin xyz="0 0 0.005" rpy="0 0 ${M_PI}"/>
-  </xacro:barret_hand>
- -->
-  <xacro:barret_hand prefix="floating" parent="floating_gripper_base" with_optoforce="False">
-    <origin xyz="0 0 0" rpy="0 0 0"/>
-  </xacro:barret_hand>
 </robot>

File: velma_moveit_config/config/velma.ros2_control.xacro (robot description, xacro)
@@ -6,5 +6,6 @@
             <hardware>
                 <!-- By default, set up controllers for simulation. This won't work on real hardware -->
-                <plugin>mock_components/GenericSystem</plugin>
+                <!-- <plugin>mock_components/GenericSystem</plugin> -->
+                <plugin>gz_ros2_control/GazeboSimSystem</plugin>
             </hardware>
             <joint name="torso_0_joint">

File: velma_moveit_config/config/velma.urdf.xacro (robot description, xacro)
@@ -6,4 +6,14 @@
     <!-- Import control_xacro -->
     <xacro:include filename="velma.ros2_control.xacro" />
+    <gazebo>
     <xacro:velma_ros2_control name="FakeSystem" initial_positions_file="$(arg initial_positions_file)"/>
+    </gazebo>
+    <xacro:velma_ros2_control name="FakeSystem" initial_positions_file="$(arg initial_positions_file)"/>
+    <gazebo>
+        <plugin filename="libgz_ros2_control-system.so"
+            name="gz_ros2_control::GazeboSimROS2ControlPlugin">
+            <parameters>$(find velma_moveit_config)/config/ros2_controllers.yaml</parameters>
+            <controller_manager_name>controller_manager</controller_manager_name>
+        </plugin>
+    </gazebo>
 </robot>
