Commit message: gravity compensation is on by default

File: velma_description/urdf/hand/barret_hand.urdf.xacro (robot description, xacro)
@@ -34,4 +34,6 @@
   <xacro:arg name="collision_model_enlargement" default="0.0"/>
   <xacro:arg name="collision_model_no_hands" default="false"/>
+  <xacro:arg name="gravity_compensation" default="true"/>
+  <xacro:property name="gravity_compensation" value="$(arg gravity_compensation)"/>
   <xacro:property name="homeDirectory" value="package://velma_description" />
   <!-- <xacro:property name="highResModelDirectory" value="${homeDirectory}/meshes/splitModels" /> -->
@@ -131,5 +133,5 @@
     </link>
     <gazebo reference="${prefix}_HandPalmLink">
-      <turnGravityOff>false</turnGravityOff>
+      <turnGravityOff>${gravity_compensation}</turnGravityOff>
       <selfCollide>true</selfCollide>
       <material>Gazebo/Blue</material>
@@ -199,5 +201,5 @@
     </link>
     <gazebo reference="${prefix}_HandGripLink">
-      <turnGravityOff>false</turnGravityOff>
+      <turnGravityOff>${gravity_compensation}</turnGravityOff>
       <selfCollide>true</selfCollide>
     </gazebo>
@@ -262,5 +264,5 @@
     </link>
     <gazebo reference="${prefix}_HandFinger${number}KnuckleOneLink">
-      <turnGravityOff>false</turnGravityOff>
+      <turnGravityOff>${gravity_compensation}</turnGravityOff>
       <selfCollide>true</selfCollide>
       <material>Gazebo/Grey</material>
@@ -344,5 +346,5 @@
     </link>
     <gazebo reference="${prefix}_HandFinger${number}KnuckleTwoLink">
-      <turnGravityOff>false</turnGravityOff>
+      <turnGravityOff>${gravity_compensation}</turnGravityOff>
       <selfCollide>true</selfCollide>
       <material>Gazebo/Grey</material>
@@ -444,5 +446,5 @@
     </link>
     <gazebo reference="${prefix}_HandFinger${number}KnuckleThreeLink">
-      <turnGravityOff>false</turnGravityOff>
+      <turnGravityOff>${gravity_compensation}</turnGravityOff>
       <selfCollide>true</selfCollide>
       <material>Gazebo/Grey</material>
@@ -505,5 +507,5 @@
         </gazebo>
         <gazebo reference="${prefix}_HandFinger${number}KnuckleThreeOptoforceSensor">
-          <turnGravityOff>false</turnGravityOff>
+          <turnGravityOff>${gravity_compensation}</turnGravityOff>
           <selfCollide>true</selfCollide>
         </gazebo>

File: velma_description/urdf/head/head.urdf.xacro (robot description, xacro)
@@ -6,4 +6,6 @@
   <xacro:arg name="collision_detector" default="fcl"/>
   <xacro:property name="collision_detector" value="$(arg collision_detector)"/>
+  <xacro:arg name="gravity_compensation" default="true"/>
+  <xacro:property name="gravity_compensation" value="$(arg gravity_compensation)"/>
   <xacro:include filename="camera.urdf.xacro" />
   <xacro:macro name="velma_head" params="parent *origin">
@@ -114,5 +116,5 @@
     </link>
     <gazebo reference="head_pan_link">
-      <turnGravityOff>false</turnGravityOff>
+      <turnGravityOff>${gravity_compensation}</turnGravityOff>
       <selfCollide>true</selfCollide>
     </gazebo>
@@ -201,10 +203,10 @@
     </link>
     <gazebo reference="head_tilt_link">
-      <turnGravityOff>false</turnGravityOff>
+      <turnGravityOff>${gravity_compensation}</turnGravityOff>
       <selfCollide>true</selfCollide>
        <material>Gazebo/DarkGrey</material>
     </gazebo>
     <gazebo reference="head_tilt_link_dummy">
-      <turnGravityOff>false</turnGravityOff>
+      <turnGravityOff>${gravity_compensation}</turnGravityOff>
       <selfCollide>true</selfCollide>
        <material>Gazebo/DarkGrey</material>

File: velma_description/urdf/torso/torso.urdf.xacro (robot description, xacro)
@@ -6,4 +6,6 @@
   <xacro:arg name="collision_detector" default="fcl"/>
   <xacro:property name="collision_detector" value="$(arg collision_detector)"/>
+  <xacro:arg name="gravity_compensation" default="true"/>
+  <xacro:property name="gravity_compensation" value="$(arg gravity_compensation)"/>
   <xacro:macro name="velma_torso" params="*origin">
     <link name="world" />
@@ -78,5 +80,5 @@
     </link>
     <gazebo reference="torso_base">
-      <turnGravityOff>false</turnGravityOff>
+      <turnGravityOff>${gravity_compensation}</turnGravityOff>
       <selfCollide>true</selfCollide>
       <material>
@@ -155,5 +157,5 @@
     </link>
     <gazebo reference="torso_link0">
-      <turnGravityOff>false</turnGravityOff>
+      <turnGravityOff>${gravity_compensation}</turnGravityOff>
       <selfCollide>true</selfCollide>
       <material>Gazebo/DarkGrey</material>
@@ -184,5 +186,5 @@
     </link>
     <gazebo reference="head_bounding_sphere">
-      <turnGravityOff>false</turnGravityOff>
+      <turnGravityOff>${gravity_compensation}</turnGravityOff>
       <selfCollide>true</selfCollide>
       <material>Gazebo/DarkGrey</material>

File: velma_description/urdf/velma.urdf.xacro (robot description, xacro)
@@ -8,4 +8,6 @@
     <selfCollide>true</selfCollide>
   </gazebo>
+  <xacro:arg name="gravity_compensation" default="true"/>
+  <xacro:property name="gravity_compensation" value="$(arg gravity_compensation)"/>
   <xacro:arg name="collision_model_full" default="false"/>
   <xacro:arg name="collision_model_simplified" default="true"/>
@@ -270,8 +272,10 @@
   </xacro:velma_torso>
   <xacro:kuka_lwr_arm parent="torso_link0" name="right" right="1">
-    <origin xyz="${cal_torso_link2_right_arm_base_joint_x} ${cal_torso_link2_right_arm_base_joint_y} ${cal_torso_link2_right_arm_base_joint_z}" rpy="${cal_torso_link2_right_arm_base_joint_roll} ${cal_torso_link2_right_arm_base_joint_pitch} ${cal_torso_link2_right_arm_base_joint_yaw}"/>
+    <origin xyz="${cal_torso_link2_right_arm_base_joint_x} ${cal_torso_link2_right_arm_base_joint_y} ${cal_torso_link2_right_arm_base_joint_z}"
+            rpy="${cal_torso_link2_right_arm_base_joint_roll} ${cal_torso_link2_right_arm_base_joint_pitch} ${cal_torso_link2_right_arm_base_joint_yaw}"/>
   </xacro:kuka_lwr_arm>
   <xacro:kuka_lwr_arm parent="torso_link0" name="left" right="1">
-    <origin xyz="${cal_torso_link2_left_arm_base_joint_x} ${cal_torso_link2_left_arm_base_joint_y} ${cal_torso_link2_left_arm_base_joint_z}" rpy="${cal_torso_link2_left_arm_base_joint_roll} ${cal_torso_link2_left_arm_base_joint_pitch} ${cal_torso_link2_left_arm_base_joint_yaw}"/>
+    <origin xyz="${cal_torso_link2_left_arm_base_joint_x} ${cal_torso_link2_left_arm_base_joint_y} ${cal_torso_link2_left_arm_base_joint_z}"
+            rpy="${cal_torso_link2_left_arm_base_joint_roll} ${cal_torso_link2_left_arm_base_joint_pitch} ${cal_torso_link2_left_arm_base_joint_yaw}"/>
   </xacro:kuka_lwr_arm>
   <joint name="right_gripper_mount_joint" type="fixed">
@@ -401,5 +405,5 @@
 -->
   <gazebo reference="right_gripper_mount_link">
-    <turnGravityOff>false</turnGravityOff>
+    <turnGravityOff>${gravity_compensation}</turnGravityOff>
     <selfCollide>true</selfCollide>
   </gazebo>
@@ -478,5 +482,5 @@
   </link>
   <gazebo reference="left_gripper_mount_link">
-    <turnGravityOff>false</turnGravityOff>
+    <turnGravityOff>${gravity_compensation}</turnGravityOff>
     <selfCollide>true</selfCollide>
   </gazebo>
@@ -489,5 +493,5 @@
   </link>
   <gazebo reference="right_FtSensorLink">
-    <turnGravityOff>false</turnGravityOff>
+    <turnGravityOff>${gravity_compensation}</turnGravityOff>
     <selfCollide>true</selfCollide>
   </gazebo>
@@ -516,5 +520,5 @@
   </link>
   <gazebo reference="left_FtSensorLink">
-    <turnGravityOff>false</turnGravityOff>
+    <turnGravityOff>${gravity_compensation}</turnGravityOff>
     <selfCollide>true</selfCollide>
   </gazebo>
@@ -600,5 +604,5 @@
   </link>
   <gazebo reference="right_keepUprightLink1">
-    <turnGravityOff>false</turnGravityOff>
+    <turnGravityOff>${gravity_compensation}</turnGravityOff>
     <selfCollide>true</selfCollide>
   </gazebo>
@@ -619,5 +623,5 @@
   </link>
   <gazebo reference="right_keepUprightLink2">
-    <turnGravityOff>false</turnGravityOff>
+    <turnGravityOff>${gravity_compensation}</turnGravityOff>
     <selfCollide>true</selfCollide>
   </gazebo>
@@ -638,5 +642,5 @@
   </link>
   <gazebo reference="left_keepUprightLink1">
-    <turnGravityOff>false</turnGravityOff>
+    <turnGravityOff>${gravity_compensation}</turnGravityOff>
     <selfCollide>true</selfCollide>
   </gazebo>
@@ -657,5 +661,5 @@
   </link>
   <gazebo reference="left_keepUprightLink2">
-    <turnGravityOff>false</turnGravityOff>
+    <turnGravityOff>${gravity_compensation}</turnGravityOff>
     <selfCollide>true</selfCollide>
   </gazebo>
