Commit message: gripper controllers

File: velma_description/urdf/hand/barret_hand.urdf.xacro (robot description, xacro)
@@ -275,5 +275,5 @@
       <origin xyz="${xyz}" rpy="${rpy}"/>
       <axis xyz="${axis}"/>
-      <limit effort="20" lower="0" upper="${PI}" velocity="3.27"/>
+      <limit effort="20" lower="-0.01" upper="${PI}" velocity="3.27"/>
       <dynamics damping="0.1"/>
     </joint>
@@ -358,5 +358,5 @@
       <axis xyz="0 0 -1"/>
                       <!-- 122 degrees - start orientation of 0.4 degrees-->
-      <limit effort="20" lower="0" upper="2.443388889" velocity="3.27"/>
+      <limit effort="20" lower="-0.01" upper="2.443388889" velocity="3.27"/>
       <dynamics damping="0.05"/>
     </joint>
@@ -459,5 +459,5 @@
       <axis xyz="0 0 -1"/>
                           <!-- measured max angle is 94.  so upper limit is 94 - start orientation (42 degrees)-->
-      <limit effort="20" lower="0" upper="0.837733333" velocity="3.27"/>
+      <limit effort="20" lower="-0.01" upper="0.837733333" velocity="3.27"/>
       <dynamics damping="0.05"/>
     </joint>

File: velma_moveit_config/config/velma.ros2_control.xacro (robot description, xacro)
@@ -174,96 +174,128 @@
                 <command_interface name="position"/>
                 <command_interface name="velocity"/>
-                <state_interface name="position"/>
-                <state_interface name="velocity"/>
+                <command_interface name="effort"/>
+                <state_interface name="position"/>
+                <state_interface name="velocity"/>
+                <state_interface name="effort"/>
             </joint>
             <joint name="left_HandFingerOneKnuckleTwoJoint">
                 <command_interface name="position"/>
                 <command_interface name="velocity"/>
-                <state_interface name="position"/>
-                <state_interface name="velocity"/>
+                <command_interface name="effort"/>
+                <state_interface name="position"/>
+                <state_interface name="velocity"/>
+                <state_interface name="effort"/>
             </joint>
             <joint name="left_HandFingerOneKnuckleThreeJoint">
                 <command_interface name="position"/>
                 <command_interface name="velocity"/>
-                <state_interface name="position"/>
-                <state_interface name="velocity"/>
+                <command_interface name="effort"/>
+                <state_interface name="position"/>
+                <state_interface name="velocity"/>
+                <state_interface name="effort"/>
             </joint>
             <joint name="left_HandFingerThreeKnuckleTwoJoint">
                 <command_interface name="position"/>
                 <command_interface name="velocity"/>
-                <state_interface name="position"/>
-                <state_interface name="velocity"/>
+                <command_interface name="effort"/>
+                <state_interface name="position"/>
+                <state_interface name="velocity"/>
+                <state_interface name="effort"/>
             </joint>
             <joint name="left_HandFingerThreeKnuckleThreeJoint">
                 <command_interface name="position"/>
                 <command_interface name="velocity"/>
-                <state_interface name="position"/>
-                <state_interface name="velocity"/>
+                <command_interface name="effort"/>
+                <state_interface name="position"/>
+                <state_interface name="velocity"/>
+                <state_interface name="effort"/>
             </joint>
             <joint name="left_HandFingerTwoKnuckleOneJoint">
                 <command_interface name="position"/>
                 <command_interface name="velocity"/>
-                <state_interface name="position"/>
-                <state_interface name="velocity"/>
+                <command_interface name="effort"/>
+                <state_interface name="position"/>
+                <state_interface name="velocity"/>
+                <state_interface name="effort"/>
             </joint>
             <joint name="left_HandFingerTwoKnuckleTwoJoint">
                 <command_interface name="position"/>
                 <command_interface name="velocity"/>
-                <state_interface name="position"/>
-                <state_interface name="velocity"/>
+                <command_interface name="effort"/>
+                <state_interface name="position"/>
+                <state_interface name="velocity"/>
+                <state_interface name="effort"/>
             </joint>
             <joint name="left_HandFingerTwoKnuckleThreeJoint">
                 <command_interface name="position"/>
                 <command_interface name="velocity"/>
-                <state_interface name="position"/>
-                <state_interface name="velocity"/>
+                <command_interface name="effort"/>
+                <state_interface name="position"/>
+                <state_interface name="velocity"/>
+                <state_interface name="effort"/>
             </joint>
             <joint name="right_HandFingerOneKnuckleOneJoint">
                 <command_interface name="position"/>
                 <command_interface name="velocity"/>
-                <state_interface name="position"/>
-                <state_interface name="velocity"/>
+                <command_interface name="effort"/>
+                <state_interface name="position"/>
+                <state_interface name="velocity"/>
+                <state_interface name="effort"/>
             </joint>
             <joint name="right_HandFingerOneKnuckleTwoJoint">
                 <command_interface name="position"/>
                 <command_interface name="velocity"/>
-                <state_interface name="position"/>
-                <state_interface name="velocity"/>
+                <command_interface name="effort"/>
+                <state_interface name="position"/>
+                <state_interface name="velocity"/>
+                <state_interface name="effort"/>
             </joint>
             <joint name="right_HandFingerOneKnuckleThreeJoint">
                 <command_interface name="position"/>
                 <command_interface name="velocity"/>
-                <state_interface name="position"/>
-                <state_interface name="velocity"/>
+                <command_interface name="effort"/>
+                <state_interface name="position"/>
+                <state_interface name="velocity"/>
+                <state_interface name="effort"/>
             </joint>
             <joint name="right_HandFingerThreeKnuckleTwoJoint">
                 <command_interface name="position"/>
                 <command_interface name="velocity"/>
-                <state_interface name="position"/>
-                <state_interface name="velocity"/>
+                <command_interface name="effort"/>
+                <state_interface name="position"/>
+                <state_interface name="velocity"/>
+                <state_interface name="effort"/>
             </joint>
             <joint name="right_HandFingerThreeKnuckleThreeJoint">
                 <command_interface name="position"/>
                 <command_interface name="velocity"/>
-                <state_interface name="position"/>
-                <state_interface name="velocity"/>
+                <command_interface name="effort"/>
+                <state_interface name="position"/>
+                <state_interface name="velocity"/>
+                <state_interface name="effort"/>
             </joint>
             <joint name="right_HandFingerTwoKnuckleOneJoint">
                 <command_interface name="position"/>
                 <command_interface name="velocity"/>
-                <state_interface name="position"/>
-                <state_interface name="velocity"/>
+                <command_interface name="effort"/>
+                <state_interface name="position"/>
+                <state_interface name="velocity"/>
+                <state_interface name="effort"/>
             </joint>
             <joint name="right_HandFingerTwoKnuckleTwoJoint">
                 <command_interface name="position"/>
                 <command_interface name="velocity"/>
-                <state_interface name="position"/>
-                <state_interface name="velocity"/>
+                <command_interface name="effort"/>
+                <state_interface name="position"/>
+                <state_interface name="velocity"/>
+                <state_interface name="effort"/>
             </joint>
             <joint name="right_HandFingerTwoKnuckleThreeJoint">
                 <command_interface name="position"/>
                 <command_interface name="velocity"/>
-                <state_interface name="position"/>
-                <state_interface name="velocity"/>
+                <command_interface name="effort"/>
+                <state_interface name="position"/>
+                <state_interface name="velocity"/>
+                <state_interface name="effort"/>
             </joint>
             <!-- Unused joints -->
