Commit message: improved head collision sphere

File: velma_description/urdf/torso/torso.urdf.xacro (robot description, xacro)
@@ -168,5 +168,5 @@
     <link name="head_bounding_sphere">
       <collision>
-        <origin xyz="0.04 0 1.6" rpy="0 0 0"/>
+        <origin xyz="0 0 1.6" rpy="0 0 0"/>
         <geometry>
           <sphere radius="0.23"/>
